File: rc_keychain.kicad_sch (KiCad schematic)
At the start: 0 parts

Commit message: progress dump
Other:
- added sheet rf (rf.kicad_sch)
Changed lines of the file:
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@@
+	)
+	(sheet
+		(at 209.55 74.93)
+		(size 30.48 24.13)
+		(exclude_from_sim no)
+		(in_bom yes)
+		(on_board yes)
+		(dnp no)
+		(fields_autoplaced yes)
+		(stroke
+			(width 0.1524)
+			(type solid)
+		)
+		(fill
+			(color 0 0 0 0.0000)
+		)
+		(property "Sheetname" "rf"
+			(at 209.55 74.2184 0)
+			(effects
+				(font
+					(size 1.27 1.27)
+				)
+				(justify left bottom)
+			)
+		)
+		(property "Sheetfile" "rf.kicad_sch"
+			(at 209.55 99.6446 0)
+			(effects
+				(font
+					(size 1.27 1.27)
+				)
+				(justify left top)
+			)
+		)
+		(instances
+			(project "rc_keychain"
+				(path "/c6cb5a1d-9f97-4766-8582-a9e93ed049e4"
+					(page "7")
+				)
+			)
+		)
 	)
 	(sheet
