File: usb.kicad_sch (KiCad schematic)
At the start: 7 parts, among them J1 USB4215-03-A_REVA, U4 USBLC6-2SC6, U5 USBLC6-2SC6

Commit message: save progress before refactor
Parts:
- J1: LCSC Part (none) -> C37616412
- R7, R8: LCSC Part (none) -> C25905
- TP6, TP7: now left out of the parts list
- U4, U5: LCSC Part (none) -> C2687116
Changed lines of the file:
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@@
+			)
+		)
+		(property "LCSC Part" "C37616412"
+			(at 121.92 97.79 0)
+			(effects
+				(font
+					(size 1.27 1.27)
+				)
+				(hide yes)
 			)
 		)
@@
 			)
 		)
+		(property "LCSC Part" "C2687116"
+			(at 184.15 114.3 0)
+			(effects
+				(font
+					(size 1.27 1.27)
+				)
+				(hide yes)
+			)
+		)
 		(pin "5"
 		)
@@
 		(unit 1)
 		(exclude_from_sim no)
-		(in_bom yes)
+		(in_bom no)
 		(on_board yes)
 		(dnp no)
@@
 		(unit 1)
 		(exclude_from_sim no)
-		(in_bom yes)
+		(in_bom no)
 		(on_board yes)
 		(dnp no)
@@
 			)
 		)
+		(property "LCSC Part" "C25905"
+			(at 87.63 92.71 90)
+			(effects
+				(font
+					(size 1.27 1.27)
+				)
+				(hide yes)
+			)
+		)
 		(pin "2"
 		)
@@
 			)
 		)
+		(property "LCSC Part" "C2687116"
+			(at 184.15 86.36 0)
+			(effects
+				(font
+					(size 1.27 1.27)
+				)
+				(hide yes)
+			)
+		)
 		(pin "1"
 		)
@@
 			(at 147.32 105.41 0)
 			(effects
+				(font
+					(size 1.27 1.27)
+				)
+				(hide yes)
+			)
+		)
+		(property "LCSC Part" "C25905"
+			(at 147.32 105.41 0)
+			(effects

Commit message: finish up everything but nfc
Parts:
- removed U4, U5: USBLC6-2SC6, Package_TO_SOT_SMD:SOT-23-6, symbol Power_Protection:USBLC6-2SC6
- added U4, U5: USBLC6-2P6, Package_TO_SOT_SMD:SOT-666, symbol Power_Protection:USBLC6-2P6
Connections:
- net +3V3: now also U5.5 (VBUS)
- net DBG_A: now also U5.6 (I/O1)
- net DBG_A_IN: now also U5.1 (I/O1)
- net DBG_B: now also U5.4 (I/O2)
- net DBG_B_IN: now also U5.3 (I/O2)
- net GND: now also J1.SH1 (SHIELD), J1.SH2 (SHIELD), J1.SH3 (SHIELD), J1.SH4 (SHIELD), U4.2 (GND), U5.2 (GND)
- net USB_DM: now also U4.4 (I/O2)
- net USB_DP: now also U4.6 (I/O1)
- net USB_IN_DM: now also U4.3 (I/O2)
- net USB_IN_DP: now also U4.1 (I/O1)
- net VBUS: now also U4.5 (VBUS)
- no-connect marks 1 -> 0
Changed lines of the file:
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@@
 	(generator_version "9.0")
 	(paper "A4")
-	(no_connect
-		(at 104.14 110.49)
+	(junction
+		(at 100.33 110.49)
+		(diameter 0)
+		(color 0 0 0 0)
+	)
+	(wire
+		(pts
+			(xy 100.33 113.03) (xy 100.33 110.49)
+		)
+		(stroke
+			(width 0)
+			(type default)
+		)
 	)
 	(wire
@@
 		(pts
 			(xy 92.71 100.33) (xy 104.14 100.33)
+		)
+		(stroke
+			(width 0)
+			(type default)
+		)
+	)
+	(wire
+		(pts
+			(xy 100.33 110.49) (xy 104.14 110.49)
 		)
 		(stroke
@@
 	)
 	(symbol
-		(lib_id "Power_Protection:USBLC6-2SC6")
+		(lib_id "Power_Protection:USBLC6-2P6")
+		(at 184.15 86.36 0)
+		(unit 1)
+		(exclude_from_sim no)
+		(in_bom yes)
+		(on_board yes)
+		(dnp no)
+		(fields_autoplaced yes)
+		(property "Reference" "U4"
+			(at 185.8011 78.74 0)
+			(effects
+				(font
+					(size 1.27 1.27)
+				)
+				(justify left)
+			)
+		)
+		(property "Value" "USBLC6-2P6"
+			(at 185.8011 81.28 0)
+			(effects
+				(font
+					(size 1.27 1.27)
+				)
+				(justify left)
+			)
+		)
+		(property "Footprint" "Package_TO_SOT_SMD:SOT-666"
+			(at 185.166 93.091 0)
+			(effects
+				(font
+					(size 1.27 1.27)
+					(italic yes)
+				)
+				(justify left)
+				(hide yes)
+			)
+		)
+		(property "Datasheet" "https://www.st.com/resource/en/datasheet/usblc6-2.pdf"
+			(at 185.166 94.996 0)
+			(effects
+				(font
+					(size 1.27 1.27)
+				)
+				(justify left)
+				(hide yes)
+			)
+		)
+		(property "Description" "Very low capacitance ESD protection diode, 2 data-line, SOT-666"
+			(at 184.15 86.36 0)
+			(effects
+				(font
+					(size 1.27 1.27)
+				)
+				(hide yes)
+			)
+		)
+		(property "LCSC Part" "C15999"
+			(at 184.15 86.36 0)
+			(effects
+				(font
+					(size 1.27 1.27)
+				)
+				(hide yes)
+			)
+		)
+		(pin "1"
+		)
+		(pin "3"
+		)
+		(pin "4"
+		)
+		(pin "2"
+		)
+		(pin "6"
+		)
+		(pin "5"
+		)
+		(instances
+			(project ""
+				(path "/c6cb5a1d-9f97-4766-8582-a9e93ed049e4/69f5d0af-289d-4671-84fe-e5e630f97c44"
+					(reference "U4")
+					(unit 1)
+				)
+			)
+		)
+	)
+	(symbol
+		(lib_id "Power_Protection:USBLC6-2P6")
 		(at 184.15 114.3 0)
 		(unit 1)
@@
 		(on_board yes)
 		(dnp no)
+		(fields_autoplaced yes)
 		(property "Reference" "U5"
-			(at 187.198 107.188 0)
-			(effects
-				(font
-					(size 1.27 1.27)
-				)
-				(justify left)
-			)
-		)
-		(property "Value" "USBLC6-2SC6"
-			(at 187.198 109.728 0)
-			(effects
-				(font
-					(size 1.27 1.27)
-				)
-				(justify left)
-			)
-		)
-		(property "Footprint" "Package_TO_SOT_SMD:SOT-23-6"
-			(at 185.42 120.65 0)
+			(at 185.8011 106.68 0)
+			(effects
+				(font
+					(size 1.27 1.27)
+				)
+				(justify left)
+			)
+		)
+		(property "Value" "USBLC6-2P6"
+			(at 185.8011 109.22 0)
+			(effects
+				(font
+					(size 1.27 1.27)
+				)
+				(justify left)
+			)
+		)
+		(property "Footprint" "Package_TO_SOT_SMD:SOT-666"
+			(at 185.166 121.031 0)
 			(effects
 				(font
@@
 		)
 		(property "Datasheet" "https://www.st.com/resource/en/datasheet/usblc6-2.pdf"
-			(at 185.42 122.555 0)
-			(effects
-				(font
-					(size 1.27 1.27)
-				)
-				(justify left)
-				(hide yes)
-			)
-		)
-		(property "Description" "Very low capacitance ESD protection diode, 2 data-line, SOT-23-6"
+			(at 185.166 122.936 0)
+			(effects
+				(font
+					(size 1.27 1.27)
+				)
+				(justify left)
+				(hide yes)
+			)
+		)
+		(property "Description" "Very low capacitance ESD protection diode, 2 data-line, SOT-666"
 			(at 184.15 114.3 0)
 			(effects
@@
 			)
 		)
-		(property "LCSC Part" "C2687116"
+		(property "LCSC Part" "C15999"
 			(at 184.15 114.3 0)
 			(effects
@@
 			)
 		)
+		(pin "2"
+		)
+		(pin "1"
+		)
 		(pin "5"
 		)
-		(pin "1"
+		(pin "6"
 		)
 		(pin "3"
 		)
-		(pin "2"
-		)
-		(pin "6"
-		)
 		(pin "4"
 		)
 		(instances
-			(project "rc_keychain"
+			(project ""
 				(path "/c6cb5a1d-9f97-4766-8582-a9e93ed049e4/69f5d0af-289d-4671-84fe-e5e630f97c44"
 					(reference "U5")
@@
 	(symbol
 		(lib_id "power:GND")
-		(at 100.33 110.49 0)
+		(at 100.33 113.03 0)
 		(unit 1)
 		(exclude_from_sim no)
@@
 		(fields_autoplaced yes)
 		(property "Reference" "#PWR020"
-			(at 100.33 116.84 0)
+			(at 100.33 119.38 0)
 			(effects
 				(font
@@
 		)
 		(property "Value" "GND"
-			(at 100.33 115.57 0)
+			(at 100.33 118.11 0)
 			(effects
 				(font
@@
 		)
 		(property "Footprint" ""
-			(at 100.33 110.49 0)
+			(at 100.33 113.03 0)
 			(effects
 				(font
@@
 		)
 		(property "Datasheet" ""
-			(at 100.33 110.49 0)
+			(at 100.33 113.03 0)
 			(effects
 				(font
@@
 		)
 		(property "Description" "Power symbol creates a global label with name \"GND\" , ground"
-			(at 100.33 110.49 0)
+			(at 100.33 113.03 0)
 			(effects
 				(font
@@
 					(unit 1)
 				)
-			)
-		)
-	)
-	(symbol
-		(lib_id "Power_Protection:USBLC6-2SC6")
-		(at 184.15 86.36 0)
-		(unit 1)
-		(exclude_from_sim no)
-		(in_bom yes)
-		(on_board yes)
-		(dnp no)
-		(property "Reference" "U4"
-			(at 185.8011 78.74 0)
-			(effects
-				(font
-					(size 1.27 1.27)
-				)
-				(justify left)
-			)
-		)
-		(property "Value" "USBLC6-2SC6"
-			(at 185.8011 81.28 0)
-			(effects
-				(font
-					(size 1.27 1.27)
-				)
-				(justify left)
-			)
-		)
-		(property "Footprint" "Package_TO_SOT_SMD:SOT-23-6"
-			(at 185.42 92.71 0)
-			(effects
-				(font
-					(size 1.27 1.27)
-					(italic yes)
-				)
-				(justify left)
-				(hide yes)
-			)
-		)
-		(property "Datasheet" "https://www.st.com/resource/en/datasheet/usblc6-2.pdf"
-			(at 185.42 94.615 0)
-			(effects
-				(font
-					(size 1.27 1.27)
-				)
-				(justify left)
-				(hide yes)
-			)
-		)
-		(property "Description" "Very low capacitance ESD protection diode, 2 data-line, SOT-23-6"
-			(at 184.15 86.36 0)
-			(effects
-				(font
-					(size 1.27 1.27)
-				)
-				(hide yes)
-			)
-		)
-		(property "LCSC Part" "C2687116"
-			(at 184.15 86.36 0)
-			(effects
-				(font
-					(size 1.27 1.27)
-				)
-				(hide yes)
-			)
-		)
-		(pin "1"
-		)
-		(pin "5"
-		)
-		(pin "3"
-		)
-		(pin "2"
-		)
-		(pin "6"
-		)
-		(pin "4"
-		)
-		(instances
-			(project "rc_keychain"
-				(path "/c6cb5a1d-9f97-4766-8582-a9e93ed049e4/69f5d0af-289d-4671-84fe-e5e630f97c44"
-					(reference "U4")
-					(unit 1)
-				)

Commit message: progress
Parts:
- removed J1: USB4215-03-A_REVA, USB4215-03-A:GCT_USB4215-03-A_REVA, symbol USB4215-03-A:USB4215-03-A_REVA
- added J1: TYPE-C 16PIN 2MD(073), TYPE-C-16PIN-2MD-073:USB-C-SMD_TYPE-C-6PIN-2MD-073, symbol TYPE-C-16PIN-2MD-073:TYPE-C16PIN2MD(073)
- R8: footprint Resistor_SMD:R_0402_1005Metric -> (none); LCSC Part C25905 -> (none)
Connections:
- net DBG_A_IN: now also J1.9 (SBU1)
- net DBG_B_IN: now also J1.3 (SBU2)
- net GND: now also R8.1, J1.1 (GND), J1.12 (GND), J1.13 (SHELL), J1.14 (SHELL); no longer R8.2
- net USB_IN_DN: now also J1.5 (DN2), J1.7 (DN1)
- net USB_IN_DP: now also J1.6 (DP1), J1.8 (DP2)
- net VBUS_RAW: now also J1.11 (VBUS), J1.2 (VBUS)
- net at R7.1: now also J1.4 (CC1)
- new net: J1.10 (CC2), R8.2
Other:
- moved on the sheet: R7

Commit message: push changes before removing fuel gauge
Parts:
- R8: footprint (none) -> Resistor_SMD:R_0402_1005Metric; LCSC Part (none) -> C25905
Changed lines of the file:
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@@
 			)
 		)
-		(property "Footprint" ""
+		(property "Footprint" "Resistor_SMD:R_0402_1005Metric"
 			(at 101.6 111.76 0)
 			(effects
@@
 			(at 101.6 111.76 90)
 			(effects
+				(font
+					(size 1.27 1.27)
+				)
+				(hide yes)
+			)
+		)
+		(property "LCSC Part" "C25905"
+			(at 101.6 111.76 90)
+			(effects

Commit message: hopefully final schematic before splitting out
Parts:
- renumbered J1 to J2, R7 to R8, R8 to R9, TP6 to TP12, TP7 to TP13
Changed lines of the file:
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@@
 		(dnp no)
 		(fields_autoplaced yes)
-		(property "Reference" "#PWR094"
+		(property "Reference" "#PWR046"
 			(at 146.05 88.9 0)
 			(effects
@@
 			(project ""
 				(path "/c6cb5a1d-9f97-4766-8582-a9e93ed049e4/69f5d0af-289d-4671-84fe-e5e630f97c44"
-					(reference "#PWR094")
+					(reference "#PWR046")
 					(unit 1)
 				)
@@
 		(dnp no)
 		(fields_autoplaced yes)
-		(property "Reference" "J1"
+		(property "Reference" "J2"
 			(at 128.905 81.28 0)
 			(effects
@@
 			(project ""
 				(path "/c6cb5a1d-9f97-4766-8582-a9e93ed049e4/69f5d0af-289d-4671-84fe-e5e630f97c44"
-					(reference "J1")
+					(reference "J2")
 					(unit 1)
 				)
@@
 		(dnp no)
 		(fields_autoplaced yes)
-		(property "Reference" "#PWR0116"
+		(property "Reference" "#PWR045"
 			(at 111.76 116.84 0)
 			(effects
@@
 			(project ""
 				(path "/c6cb5a1d-9f97-4766-8582-a9e93ed049e4/69f5d0af-289d-4671-84fe-e5e630f97c44"
-					(reference "#PWR0116")
+					(reference "#PWR045")
 					(unit 1)
 				)
@@
 		(dnp no)
 		(fields_autoplaced yes)
-		(property "Reference" "#PWR024"
+		(property "Reference" "#PWR048"
 			(at 184.15 85.09 0)
 			(effects
@@
 			(project "rc_keychain"
 				(path "/c6cb5a1d-9f97-4766-8582-a9e93ed049e4/69f5d0af-289d-4671-84fe-e5e630f97c44"
-					(reference "#PWR024")
+					(reference "#PWR048")
 					(unit 1)
 				)
@@
 		(dnp no)
 		(fields_autoplaced yes)
-		(property "Reference" "#PWR0119"
+		(property "Reference" "#PWR042"
 			(at 96.52 105.41 0)
 			(effects
@@
 			(project ""
 				(path "/c6cb5a1d-9f97-4766-8582-a9e93ed049e4/69f5d0af-289d-4671-84fe-e5e630f97c44"
-					(reference "#PWR0119")
+					(reference "#PWR042")
 					(unit 1)
 				)
@@
 		(dnp no)
 		(fields_autoplaced yes)
-		(property "Reference" "R8"
+		(property "Reference" "R9"
 			(at 101.6 106.68 90)
 			(effects
@@
 			(project ""
 				(path "/c6cb5a1d-9f97-4766-8582-a9e93ed049e4/69f5d0af-289d-4671-84fe-e5e630f97c44"
-					(reference "R8")
+					(reference "R9")
 					(unit 1)
 				)
@@
 		(dnp no)
 		(fields_autoplaced yes)
-		(property "Reference" "TP7"
+		(property "Reference" "TP13"
 			(at 217.17 88.8999 90)
 			(effects
@@
 			(project "rc_keychain"
 				(path "/c6cb5a1d-9f97-4766-8582-a9e93ed049e4/69f5d0af-289d-4671-84fe-e5e630f97c44"
-					(reference "TP7")
+					(reference "TP13")
 					(unit 1)
 				)
@@
 		(dnp no)
 		(fields_autoplaced yes)
-		(property "Reference" "TP6"
+		(property "Reference" "TP12"
 			(at 217.17 83.8199 90)
 			(effects
@@
 			(project "rc_keychain"
 				(path "/c6cb5a1d-9f97-4766-8582-a9e93ed049e4/69f5d0af-289d-4671-84fe-e5e630f97c44"
-					(reference "TP6")
+					(reference "TP12")
 					(unit 1)
 				)
@@
 		(dnp no)
 		(fields_autoplaced yes)
-		(property "Reference" "R7"
+		(property "Reference" "R8"
 			(at 101.6 91.44 90)
 			(effects
@@
 			(project "rc_keychain"
 				(path "/c6cb5a1d-9f97-4766-8582-a9e93ed049e4/69f5d0af-289d-4671-84fe-e5e630f97c44"
-					(reference "R7")
+					(reference "R8")
 					(unit 1)
 				)
@@
 		(dnp no)
 		(fields_autoplaced yes)
-		(property "Reference" "#PWR0118"
+		(property "Reference" "#PWR043"
 			(at 96.52 120.65 0)
 			(effects
@@
 			(project ""
 				(path "/c6cb5a1d-9f97-4766-8582-a9e93ed049e4/69f5d0af-289d-4671-84fe-e5e630f97c44"
-					(reference "#PWR0118")
+					(reference "#PWR043")
 					(unit 1)
 				)
@@
 		(dnp no)
 		(fields_autoplaced yes)
-		(property "Reference" "#PWR0115"
+		(property "Reference" "#PWR047"
 			(at 146.05 116.84 0)
 			(effects
@@
 			(project ""
 				(path "/c6cb5a1d-9f97-4766-8582-a9e93ed049e4/69f5d0af-289d-4671-84fe-e5e630f97c44"
-					(reference "#PWR0115")
+					(reference "#PWR047")
 					(unit 1)
 				)
@@
 		(on_board yes)
 		(dnp no)
-		(property "Reference" "#PWR045"
+		(property "Reference" "#PWR050"
 			(at 184.15 113.03 0)
 			(effects
@@
 			(project "rc_keychain"
 				(path "/c6cb5a1d-9f97-4766-8582-a9e93ed049e4/69f5d0af-289d-4671-84fe-e5e630f97c44"
-					(reference "#PWR045")
+					(reference "#PWR050")
 					(unit 1)
 				)
@@
 		(dnp no)
 		(fields_autoplaced yes)
-		(property "Reference" "#PWR0117"
+		(property "Reference" "#PWR044"
 			(at 111.76 88.9 0)
 			(effects
@@
 			(project ""
 				(path "/c6cb5a1d-9f97-4766-8582-a9e93ed049e4/69f5d0af-289d-4671-84fe-e5e630f97c44"
-					(reference "#PWR0117")
+					(reference "#PWR044")
 					(unit 1)
 				)
@@
 		(on_board yes)
 		(dnp no)
-		(property "Reference" "#PWR025"
+		(property "Reference" "#PWR049"
 			(at 184.15 100.33 0)
 			(effects
@@
 			(project "rc_keychain"
 				(path "/c6cb5a1d-9f97-4766-8582-a9e93ed049e4/69f5d0af-289d-4671-84fe-e5e630f97c44"
-					(reference "#PWR025")
+					(reference "#PWR049")
 					(unit 1)
 				)
@@
 		(dnp no)
 		(fields_autoplaced yes)
-		(property "Reference" "#PWR046"
+		(property "Reference" "#PWR051"
 			(at 184.15 128.27 0)
 			(effects
@@
 			(project "rc_keychain"
 				(path "/c6cb5a1d-9f97-4766-8582-a9e93ed049e4/69f5d0af-289d-4671-84fe-e5e630f97c44"
-					(reference "#PWR046")
-					(unit 1)
-				)
+					(reference "#PWR051")
+					(unit 1)
+				)

Commit message: final review, fixes, cleanup
Parts:
- TP13: value USB_DM -> USB_DN
Connections:
- net USB_IN_DM is gone; now on net USB_IN_DN: U4.3 (I/O2)
- net VBUS is gone; now on net VBUS_RAW: U4.5 (VBUS)
- net USB_DM renamed USB_DN
Changed lines of the file:
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@@
+	(wire
+		(pts
+			(xy 181.61 78.74) (xy 184.15 78.74)
+		)
+		(stroke
+			(width 0)
+			(type default)
+		)
+	)
 	(wire
 		(pts
@@
 		(pts
 			(xy 104.14 111.76) (xy 118.11 111.76)
+		)
+		(stroke
+			(width 0)
+			(type default)
+		)
+	)
+	(wire
+		(pts
+			(xy 184.15 78.74) (xy 184.15 81.28)
 		)
 		(stroke
@@
 		)
 	)
-	(label "USB_IN_DM"
+	(label "USB_IN_DN"
 		(at 167.64 88.9 0)
 		(effects
@@
 		)
 	)
-	(global_label "USB_DM"
+	(global_label "USB_DN"
 		(shape input)
 		(at 212.09 90.17 180)
@@
 		)
 		(property "Intersheetrefs" "${INTERSHEET_REFS}"
-			(at 201.6058 90.17 0)
+			(at 201.7267 90.17 0)
 			(effects
 				(font
@@
 		)
 	)
+	(global_label "VBUS_RAW"
+		(shape input)
+		(at 181.61 78.74 180)
+		(fields_autoplaced yes)
+		(effects
+			(font
+				(size 1.27 1.27)
+			)
+			(justify right)
+		)
+		(property "Intersheetrefs" "${INTERSHEET_REFS}"
+			(at 168.9486 78.74 0)
+			(effects
+				(font
+					(size 1.27 1.27)
+				)
+				(justify right)
+				(hide yes)
+			)
+		)
+	)
 	(global_label "DBG_B"
 		(shape input)
@@
 		)
 	)
-	(global_label "USB_DM"
+	(global_label "USB_DN"
 		(shape input)
 		(at 189.23 88.9 0)
@@
 		)
 		(property "Intersheetrefs" "${INTERSHEET_REFS}"
-			(at 199.7142 88.9 0)
+			(at 199.5933 88.9 0)
 			(effects
 				(font
@@
 	)
 	(symbol
-		(lib_id "power:VBUS")
-		(at 184.15 81.28 0)
-		(unit 1)
-		(exclude_from_sim no)
-		(in_bom yes)
-		(on_board yes)
-		(dnp no)
-		(fields_autoplaced yes)
-		(property "Reference" "#PWR048"
-			(at 184.15 85.09 0)
-			(effects
-				(font
-					(size 1.27 1.27)
-				)
-				(hide yes)
-			)
-		)
-		(property "Value" "VBUS"
-			(at 184.15 76.2 0)
-			(effects
-				(font
-					(size 1.27 1.27)
-				)
-			)
-		)
-		(property "Footprint" ""
-			(at 184.15 81.28 0)
-			(effects
-				(font
-					(size 1.27 1.27)
-				)
-				(hide yes)
-			)
-		)
-		(property "Datasheet" ""
-			(at 184.15 81.28 0)
-			(effects
-				(font
-					(size 1.27 1.27)
-				)
-				(hide yes)
-			)
-		)
-		(property "Description" "Power symbol creates a global label with name \"VBUS\""
-			(at 184.15 81.28 0)
-			(effects
-				(font
-					(size 1.27 1.27)
-				)
-				(hide yes)
-			)
-		)
-		(pin "1"
-		)
-		(instances
-			(project "rc_keychain"
-				(path "/c6cb5a1d-9f97-4766-8582-a9e93ed049e4/69f5d0af-289d-4671-84fe-e5e630f97c44"
-					(reference "#PWR048")
-					(unit 1)
-				)
-			)
-		)
-	)
-	(symbol
 		(lib_id "power:GND")
 		(at 96.52 99.06 0)
@@
 			)
 		)
-		(property "Value" "USB_DM"
+		(property "Value" "USB_DN"
 			(at 217.17 91.4399 90)
 			(effects
