File: rc_keychain.kicad_pcb (KiCad board)
At the start: 2 copper layers, 51.5 x 17 mm, 64 parts, among them J1 USB4215-03-A_REVA, J2 U.FL-R-SMT-1(10), J3 Touch_Top, J4 Touch_Top, SW2 TS35CA, U1 SF32LB525UC6, U2 BQ27426YZFR, U3 TPS25200DRVT, U4 USBLC6-2SC6, U5 USBLC6-2SC6, U6 GD25Q64ESIG, U7 MTCH2120-V/REB, U8 MTCH2120-V/REB, Y1 32.768khz, Y2 48MHz

Commit message: save progress before refactor
Parts:
- removed J2: U.FL-R-SMT-1(10), U.FL-R-SMT-1_10_:HRS_U.FL-R-SMT-1_10_
- removed Y1: 32.768khz, Crystal:Crystal_SMD_2520-4Pin_2.5x2.0mm
- added C26: 10uF, Capacitor_SMD:C_0402_1005Metric, F.Cu at (145.1, 134.5)
- added C27: 1uF, Capacitor_SMD:C_0402_1005Metric, F.Cu at (145.1, 136.5)
- added C28: 10uF, Capacitor_SMD:C_0402_1005Metric, F.Cu at (145.1, 138.5)
- added C29: 2.2uF, Capacitor_SMD:C_0603_1608Metric, F.Cu at (153.4, 137.6)
- added C30: 4.7uF, Capacitor_SMD:C_0402_1005Metric, F.Cu at (145.1, 140.4)
- added C31: 15pF, Capacitor_SMD:C_0402_1005Metric, F.Cu at (145.1, 142.4)
- added C32: 4.7uF, Capacitor_SMD:C_0603_1608Metric, F.Cu at (153.4, 140.1)
- added D1: MBR0520, Diode_SMD:D_SOD-123, F.Cu at (150.5, 158.5)
- added J5: 5034801200, 5034801200:CON_5034801200_MOL, F.Cu at (143.5, 155.2)
- added L4: 4.7uH, Inductor_SMD:L_1008_2520Metric, F.Cu at (154.9, 129.5)
- added R13: 100k, Resistor_SMD:R_0402_1005Metric, F.Cu at (196.0, 131.5)
- added R14: 100k, Resistor_SMD:R_0402_1005Metric, F.Cu at (196.0, 133.5)
- added R15: 100k, Resistor_SMD:R_0402_1005Metric, F.Cu at (196.0, 135.5)
- added R16: 100k, Resistor_SMD:R_0402_1005Metric, F.Cu at (196.0, 137.5)
- added R17: 100k, Resistor_SMD:R_0402_1005Metric, F.Cu at (196.0, 139.5)
- added R18: 100k, Resistor_SMD:R_0402_1005Metric, F.Cu at (196.0, 141.5)
- added R19: 100k, Resistor_SMD:R_0402_1005Metric, F.Cu at (196.2, 143.5)
- added R20: 100k, Resistor_SMD:R_0402_1005Metric, F.Cu at (198.9, 131.5)
- added R21: 100k, Resistor_SMD:R_0402_1005Metric, F.Cu at (198.9, 133.5)
- added R22: 100k, Resistor_SMD:R_0402_1005Metric, F.Cu at (198.9, 135.5)
- added R23: 100k, Resistor_SMD:R_0402_1005Metric, F.Cu at (198.9, 137.5)
- added R24: 100k, Resistor_SMD:R_0402_1005Metric, F.Cu at (198.9, 139.5)
- added R25: 100k, Resistor_SMD:R_0402_1005Metric, F.Cu at (198.9, 141.5)
- added R26: 100k, Resistor_SMD:R_0402_1005Metric, F.Cu at (199.1, 143.5)
- added R27: 100k, Resistor_SMD:R_0402_1005Metric, F.Cu at (201.8, 131.5)
- added R28: 100k, Resistor_SMD:R_0402_1005Metric, F.Cu at (201.8, 133.5)
- added R29: 100k, Resistor_SMD:R_0402_1005Metric, F.Cu at (201.8, 135.5)
- added R30: 100k, Resistor_SMD:R_0402_1005Metric, F.Cu at (201.8, 137.5)
- added R31: 100k, Resistor_SMD:R_0402_1005Metric, F.Cu at (201.8, 139.5)
- added R32: 100k, Resistor_SMD:R_0402_1005Metric, F.Cu at (201.8, 141.5)
- added R33: 100k, Resistor_SMD:R_0402_1005Metric, F.Cu at (202.0, 143.5)
- added R34: 100k, Resistor_SMD:R_0402_1005Metric, F.Cu at (204.7, 131.5)
- added R35: 100k, Resistor_SMD:R_0402_1005Metric, F.Cu at (204.7, 133.5)
- added R36: 100k, Resistor_SMD:R_0402_1005Metric, F.Cu at (204.7, 135.5)
- added R37: 100k, Resistor_SMD:R_0402_1005Metric, F.Cu at (142.3, 136.5)
- added R38: 560k, Resistor_SMD:R_0402_1005Metric, F.Cu at (148.0, 154.5)
- added R39: 820k, Resistor_SMD:R_0402_1005Metric, F.Cu at (142.3, 140.5)
- added R40: 130k, Resistor_SMD:R_0402_1005Metric, F.Cu at (142.3, 142.5)
- added TP8: SCL, TestPoint:TestPoint_Pad_1.5x1.5mm, F.Cu at (136.8, 134.9)
- added TP9: SDA, TestPoint:TestPoint_Pad_1.5x1.5mm, F.Cu at (136.8, 138.5)
- added U10: TPS61040DBV, Package_TO_SOT_SMD:SOT-23-5, F.Cu at (150.5, 161.5)
- added U9: AP3602AKTR-G1, AP3602AKTR-G1:SOT-23-6_L2.9-W1.6-P0.95-LS2.8-BR, F.Cu at (172.0, 155.5)
- C10, C6: footprint Capacitor_SMD:C_0402_1005Metric -> Capacitor_SMD:C_0603_1608Metric
- C2: value 0.47uF -> 470nF; footprint Capacitor_SMD:C_0402_1005Metric -> Capacitor_SMD:C_0603_1608Metric
- C5: value 0.1uF -> 100nF
- J4: value Touch_Top -> Touch_Btm
- L1: footprint Inductor_SMD:L_0603_1608Metric -> Inductor_SMD:L_0402_1005Metric
- R4, R5, R6: footprint Resistor_SMD:R_0402_1005Metric -> Resistor_SMD:R_0603_1608Metric
- U6: value GD25Q64ESIG -> GD25Q64CWIGR; footprint GD25Q64ESIG:SOP-8_L5.3-W5.3-P1.27-LS8.0-BL -> GD25Q64CWIGR:WSON-8_L6.0-W5.0-P1.27-BL-EP
- moved U3 63.4 mm to (131.5, 155.8)
- moved Y2 62.7 mm to (166.5, 155.0)
- moved U4 61.7 mm to (130.5, 161.0), turned to 90 degrees
- moved R10 58.0 mm to (162.0, 158.5)
- moved C15 52.0 mm to (172.7, 140.3)
- moved C8 48.2 mm to (169.9, 136.4)
- moved C9 48.2 mm to (169.9, 138.4)
- moved C11 46.3 mm to (169.9, 140.3)
- moved C1 46.3 mm to (167.0, 134.4)
- moved C16 45.4 mm to (175.6, 134.4)
- moved C18 45.4 mm to (175.6, 138.4)
- moved C19 45.4 mm to (175.6, 140.3)
- moved U5 45.2 mm to (134.9, 147.9), turned to 180 degrees
- moved R2 45.2 mm to (163.5, 149.5), turned to -90 degrees
- moved C3 44.4 mm to (167.0, 136.4)
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Connections:
- J4 pad 1: unconnected-(J4-Pin_1-Pad1) -> /touch/TOUCH_BTM_1
- J4 pad 10: unconnected-(J4-Pin_10-Pad10) -> /touch/TOUCH_BTM_10
- J4 pad 11: unconnected-(J4-Pin_11-Pad11) -> /touch/TOUCH_BTM_11
- J4 pad 12: unconnected-(J4-Pin_12-Pad12) -> /touch/TOUCH_BTM_12
- J4 pad 2: unconnected-(J4-Pin_2-Pad2) -> /touch/TOUCH_BTM_2
- J4 pad 3: unconnected-(J4-Pin_3-Pad3) -> /touch/TOUCH_BTM_3
- J4 pad 4: unconnected-(J4-Pin_4-Pad4) -> /touch/TOUCH_BTM_4
- J4 pad 5: unconnected-(J4-Pin_5-Pad5) -> /touch/TOUCH_BTM_5
- J4 pad 6: unconnected-(J4-Pin_6-Pad6) -> /touch/TOUCH_BTM_6
- J4 pad 7: unconnected-(J4-Pin_7-Pad7) -> /touch/TOUCH_BTM_7
- J4 pad 8: unconnected-(J4-Pin_8-Pad8) -> /touch/TOUCH_BTM_8
- J4 pad 9: unconnected-(J4-Pin_9-Pad9) -> /touch/TOUCH_BTM_9
- LED1 pad 2: unconnected-(LED1-GND-Pad2) -> GND
- LED1 pad 3: unconnected-(LED1-SDI-Pad3) -> LED_DAT
- LED1 pad 4: unconnected-(LED1-CKL-Pad4) -> LED_CLK
- LED1 pad 5: unconnected-(LED1-VDD-Pad5) -> +5V
- U1 pad 25: unconnected-(U1B-PA20-Pad25) -> HAPTIC_PWM
- U1 pad 49: unconnected-(U1B-PA2-Pad49) -> OLED_EN
- U1 pad 5: unconnected-(U1B-PA28-Pad5) -> LED_CLK
- U1 pad 6: unconnected-(U1B-PA27-Pad6) -> LED_EN
- U1 pad 9: unconnected-(U1B-PA24-Pad9) -> LED_DAT
- U7 pad 10: unconnected-(U7-BUTTON5/GPIO5-Pad10) -> Net-(U7-BUTTON5/GPIO5)
- U7 pad 13: unconnected-(U7-BUTTON6/GPIO6-Pad13) -> Net-(U7-BUTTON6/GPIO6)
- U7 pad 14: unconnected-(U7-BUTTON7/GPIO7-Pad14) -> Net-(U7-BUTTON7/GPIO7)
- U7 pad 15: unconnected-(U7-BUTTON8/GPIO8-Pad15) -> Net-(U7-BUTTON8/GPIO8)
- U7 pad 16: unconnected-(U7-BUTTON9/GPIO9-Pad16) -> Net-(U7-BUTTON9/GPIO9)
- U7 pad 17: unconnected-(U7-BUTTON10/GPIO10-Pad17) -> Net-(U7-BUTTON10/GPIO10)
- U7 pad 18: unconnected-(U7-BUTTON11/DS/GPIO11-Pad18) -> Net-(U7-BUTTON11/DS/GPIO11)
- U7 pad 2: unconnected-(U7-ADD_SEL-Pad2) -> GND
- U7 pad 5: unconnected-(U7-BUTTON0/GPIO0-Pad5) -> Net-(U7-BUTTON0/GPIO0)
- U7 pad 6: unconnected-(U7-BUTTON1/GPIO1-Pad6) -> Net-(U7-BUTTON1/GPIO1)
- U7 pad 7: unconnected-(U7-BUTTON2/GPIO2-Pad7) -> Net-(U7-BUTTON2/GPIO2)
- U7 pad 8: unconnected-(U7-BUTTON3/GPIO3-Pad8) -> Net-(U7-BUTTON3/GPIO3)
- U7 pad 9: unconnected-(U7-BUTTON4/GPIO4-Pad9) -> Net-(U7-BUTTON4/GPIO4)
- U8 pad 10: unconnected-(U8-BUTTON5/GPIO5-Pad10) -> Net-(U8-BUTTON5/GPIO5)
- U8 pad 13: unconnected-(U8-BUTTON6/GPIO6-Pad13) -> Net-(U8-BUTTON6/GPIO6)
- U8 pad 14: unconnected-(U8-BUTTON7/GPIO7-Pad14) -> Net-(U8-BUTTON7/GPIO7)
- U8 pad 15: unconnected-(U8-BUTTON8/GPIO8-Pad15) -> Net-(U8-BUTTON8/GPIO8)
- U8 pad 16: unconnected-(U8-BUTTON9/GPIO9-Pad16) -> Net-(U8-BUTTON9/GPIO9)
- U8 pad 17: unconnected-(U8-BUTTON10/GPIO10-Pad17) -> Net-(U8-BUTTON10/GPIO10)
- U8 pad 18: unconnected-(U8-BUTTON11/DS/GPIO11-Pad18) -> Net-(U8-BUTTON11/DS/GPIO11)
- U8 pad 5: unconnected-(U8-BUTTON0/GPIO0-Pad5) -> Net-(U8-BUTTON0/GPIO0)
- U8 pad 6: unconnected-(U8-BUTTON1/GPIO1-Pad6) -> Net-(U8-BUTTON1/GPIO1)
- U8 pad 7: unconnected-(U8-BUTTON2/GPIO2-Pad7) -> Net-(U8-BUTTON2/GPIO2)
- U8 pad 8: unconnected-(U8-BUTTON3/GPIO3-Pad8) -> Net-(U8-BUTTON3/GPIO3)
- U8 pad 9: unconnected-(U8-BUTTON4/GPIO4-Pad9) -> Net-(U8-BUTTON4/GPIO4)
Other:
- board size 51.5 x 17 mm -> 58 x 18 mm

Commit message: progress dump
Parts:
- moved R33 31.9 mm to (174.6, 159.8)
- moved R26 31.6 mm to (174.5, 163.4)
- moved R18 29.9 mm to (174.5, 162.2)
- moved R19 27.9 mm to (174.5, 161.0)
Changed lines of the file:
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@@
 	(footprint "Resistor_SMD:R_0402_1005Metric"
 		(layer "F.Cu")
-		(at 196.19 143.5)
+		(at 174.51 161)
 		(descr "Resistor SMD 0402 (1005 Metric), square (rectangular) end terminal, IPC-7351 nominal, (Body size source: IPC-SM-782 page 72, https://www.pcb-3d.com/wordpress/wp-content/uploads/ipc-sm-782a_amendment_1_and_2.pdf), generated with kicad-footprint-generator")
 		(tags "resistor")
@@
 	(footprint "Resistor_SMD:R_0402_1005Metric"
 		(layer "F.Cu")
-		(at 195.99 141.47)
+		(at 174.51 162.2)
 		(descr "Resistor SMD 0402 (1005 Metric), square (rectangular) end terminal, IPC-7351 nominal, (Body size source: IPC-SM-782 page 72, https://www.pcb-3d.com/wordpress/wp-content/uploads/ipc-sm-782a_amendment_1_and_2.pdf), generated with kicad-footprint-generator")
 		(tags "resistor")
@@
 	(footprint "Resistor_SMD:R_0402_1005Metric"
 		(layer "F.Cu")
-		(at 202.01 143.5)
+		(at 174.6 159.8)
 		(descr "Resistor SMD 0402 (1005 Metric), square (rectangular) end terminal, IPC-7351 nominal, (Body size source: IPC-SM-782 page 72, https://www.pcb-3d.com/wordpress/wp-content/uploads/ipc-sm-782a_amendment_1_and_2.pdf), generated with kicad-footprint-generator")
 		(tags "resistor")
@@
 	(footprint "Resistor_SMD:R_0402_1005Metric"
 		(layer "F.Cu")
-		(at 199.1 143.5)
+		(at 174.51 163.4)
 		(descr "Resistor SMD 0402 (1005 Metric), square (rectangular) end terminal, IPC-7351 nominal, (Body size source: IPC-SM-782 page 72, https://www.pcb-3d.com/wordpress/wp-content/uploads/ipc-sm-782a_amendment_1_and_2.pdf), generated with kicad-footprint-generator")
 		(tags "resistor")

Commit message: finish up everything but nfc
Parts:
- removed U6: GD25Q64CWIGR, GD25Q64CWIGR:WSON-8_L6.0-W5.0-P1.27-BL-EP
- added C33: 4.7nF, Capacitor_SMD:C_0402_1005Metric, F.Cu at (180.4, 113.9)
- added D2: BAT54WS, Diode_SMD:D_SOD-323F, F.Cu at (180.2, 117.8)
- added D3: BZT52B3V3, Diode_SMD:D_SOD-123, F.Cu at (176.1, 114.6)
- added J2: U.FL-R-SMT-1(10), U.FL-R-SMT-1_10_:HRS_U.FL-R-SMT-1_10_, F.Cu at (175.9, 125.0)
- added Q1: 2N7002, Package_TO_SOT_SMD:SOT-23, F.Cu at (175.6, 118.7)
- added R45: 4.7k, Resistor_SMD:R_0402_1005Metric, F.Cu at (180.2, 123.9)
- added R46: 4.7k, Resistor_SMD:R_0402_1005Metric, F.Cu at (180.2, 125.9)
- added REF**: WSON-8-1EP_8x6mm_P1.27mm_EP3.4x4.3mm, Package_SON:WSON-8-1EP_8x6mm_P1.27mm_EP3.4x4.3mm, F.Cu at (156.6, 160.2)
- LED1: value SK9822-EC20 -> XL-4020RGBC-WS2812B; footprint SK9822-EC20:LED-SMD_6P-L2.0-W2.0-P0.80-TL -> XL-4020RGBC-2812B:LED-SMD_4P-L4.0-W1.7_XL-4020RGBC-WS2812B
- R10, R9: value 10k -> 4.7k
- TP8: value SCL -> SCL_G1
- TP9: value SDA -> SDA_G1
- moved SW2 47.1 mm to (131.0, 162.4), turned to 180 degrees
- moved LED1 40.9 mm to (136.1, 162.7)
- moved R36 40.5 mm to (174.8, 162.8)
- moved R35 40.2 mm to (177.1, 162.7)
- moved R32 38.2 mm to (169.9, 162.4)
- moved R34 37.5 mm to (172.2, 150.2)
- moved R31 37.2 mm to (172.7, 162.6)
- moved R30 37.0 mm to (171.4, 158.6)
- moved R29 36.9 mm to (171.5, 156.5)
- moved R27 36.7 mm to (171.5, 152.2)
- moved U9 35.7 mm to (136.4, 157.8)
- moved R28 35.2 mm to (171.4, 151.2)
- moved R20 35.1 mm to (171.4, 153.3)
- moved R24 34.2 mm to (171.5, 159.9)
- moved R21 34.1 mm to (171.8, 154.3)
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Connections:
- J1 pad SH1: unconnected-(J1-SHIELD-PadSH1)_1 -> GND
- J1 pad SH2: unconnected-(J1-SHIELD-PadSH1)_2 -> GND
- J1 pad SH3: unconnected-(J1-SHIELD-PadSH1)_3 -> GND
- J1 pad SH4: unconnected-(J1-SHIELD-PadSH1) -> GND
- J3 pad 1: unconnected-(J3-Pin_1-Pad1) -> /touch/TOUCH_TOP_1
- J3 pad 10: unconnected-(J3-Pin_10-Pad10) -> /touch/TOUCH_TOP_10
- J3 pad 11: unconnected-(J3-Pin_11-Pad11) -> /touch/TOUCH_TOP_11
- J3 pad 12: unconnected-(J3-Pin_12-Pad12) -> /touch/TOUCH_TOP_12
- J3 pad 2: unconnected-(J3-Pin_2-Pad2) -> /touch/TOUCH_TOP_2
- J3 pad 3: unconnected-(J3-Pin_3-Pad3) -> /touch/TOUCH_TOP_3
- J3 pad 4: unconnected-(J3-Pin_4-Pad4) -> /touch/TOUCH_TOP_4
- J3 pad 5: unconnected-(J3-Pin_5-Pad5) -> /touch/TOUCH_TOP_5
- J3 pad 6: unconnected-(J3-Pin_6-Pad6) -> /touch/TOUCH_TOP_6
- J3 pad 7: unconnected-(J3-Pin_7-Pad7) -> /touch/TOUCH_TOP_7
- J3 pad 8: unconnected-(J3-Pin_8-Pad8) -> /touch/TOUCH_TOP_8
- J3 pad 9: unconnected-(J3-Pin_9-Pad9) -> /touch/TOUCH_TOP_9
- J5 pad 3: +3V3_G1 -> +3V3_G2
- LED1 pad 1: unconnected-(LED1-SDO-Pad1) -> +5V
- LED1 pad 2: GND -> unconnected-(LED1-DO-Pad2)
- LED1 pad 3: LED_DAT -> GND
- LED1 pad 4: LED_CLK -> LED_DAT
- R10 pad 1: SCL -> SCL_G1
- R10 pad 2: +3V3 -> +3V3_G1
- R25 pad 1: unconnected-(R25-Pad1) -> /touch/TOUCH_TOP_1
- R26 pad 1: unconnected-(R26-Pad1) -> /touch/TOUCH_TOP_2
- R27 pad 1: unconnected-(R27-Pad1) -> /touch/TOUCH_TOP_3
- R28 pad 1: unconnected-(R28-Pad1) -> /touch/TOUCH_TOP_4
- R29 pad 1: unconnected-(R29-Pad1) -> /touch/TOUCH_TOP_5
- R30 pad 1: unconnected-(R30-Pad1) -> /touch/TOUCH_TOP_6
- R31 pad 2: unconnected-(R31-Pad2) -> /touch/TOUCH_TOP_12
- R32 pad 2: unconnected-(R32-Pad2) -> /touch/TOUCH_TOP_11
- R33 pad 2: unconnected-(R33-Pad2) -> /touch/TOUCH_TOP_10
- R34 pad 2: unconnected-(R34-Pad2) -> /touch/TOUCH_TOP_9
- R35 pad 2: unconnected-(R35-Pad2) -> /touch/TOUCH_TOP_8
- R36 pad 2: unconnected-(R36-Pad2) -> /touch/TOUCH_TOP_7
- R9 pad 1: SDA -> SDA_G1
- R9 pad 2: +3V3 -> +3V3_G1
- TP8 pad 1: SCL -> SCL_G1
- TP9 pad 1: SDA -> SDA_G1
- U1 pad 1: unconnected-(U1B-PA32-Pad1) -> SDA_G1
- U1 pad 5: LED_CLK -> unconnected-(U1B-PA28-Pad5)
- U1 pad 56: unconnected-(U1B-PA44-Pad56) -> TOUCH_RST
- U1 pad 57: unconnected-(U1B-PA43-Pad57) -> TOUCH_INT
- U1 pad 67: unconnected-(U1B-PA33-Pad67) -> SCL_G1
- U7 pad 1: unconnected-(U7-SCL-Pad1) -> SCL_G1
- U7 pad 11: unconnected-(U7-INT*-Pad11) -> TOUCH_INT
- U7 pad 12: unconnected-(U7-GPIO12-Pad12) -> GND
- U7 pad 19: unconnected-(U7-RESET*-Pad19) -> TOUCH_RST
- U7 pad 20: unconnected-(U7-SDA-Pad20) -> SDA_G1
- U7 pad 21: unconnected-(U7-EPAD-Pad21) -> GND
- U7 pad 3: unconnected-(U7-GND-Pad3) -> GND
- U7 pad 4: unconnected-(U7-VDD-Pad4) -> +3V3_G1
- U8 pad 1: unconnected-(U8-SCL-Pad1) -> SCL_G1
- U8 pad 11: unconnected-(U8-INT*-Pad11) -> TOUCH_INT
- U8 pad 12: unconnected-(U8-GPIO12-Pad12) -> GND
- U8 pad 19: unconnected-(U8-RESET*-Pad19) -> TOUCH_RST
- U8 pad 2: unconnected-(U8-ADD_SEL-Pad2) -> +3V3_G1
- U8 pad 20: unconnected-(U8-SDA-Pad20) -> SDA_G1
- U8 pad 21: unconnected-(U8-EPAD-Pad21) -> GND
- U8 pad 3: unconnected-(U8-GND-Pad3) -> GND
- U8 pad 4: unconnected-(U8-VDD-Pad4) -> +3V3_G1
Other:
- outline, holes or cut-outs redrawn

Commit message: progress
Parts:
- removed J3: Touch_Top, custom_footprints:Touch_Surface_12_Pad
- removed J4: Touch_Btm, custom_footprints:Touch_Surface_12_Pad
- removed R10, R45, R46, R9: 4.7k, Resistor_SMD:R_0402_1005Metric
- removed R13, R14, R15, R16, R17, R18, R19, R20, R21, R22, R23, R24, R25, R26, R27, R28, R29, R30, R31, R32, R33, R34, R35, R36: 100k, Resistor_SMD:R_0402_1005Metric
- removed R8: 5.1k, Resistor_SMD:R_0402_1005Metric
- removed REF**: WSON-8-1EP_8x6mm_P1.27mm_EP3.4x4.3mm, Package_SON:WSON-8-1EP_8x6mm_P1.27mm_EP3.4x4.3mm
- added BT1: Battery_Cell, custom_footprints:Generic_Solder_Pads_2P, F.Cu at (159.5, 121.5)
- added C34: 10nF, Capacitor_SMD:C_0402_1005Metric, F.Cu at (147.4, 101.9)
- added C39: 100nF, Capacitor_SMD:C_0402_1005Metric, F.Cu at (146.2, 120.9)
- added C40: 10uF, Capacitor_SMD:C_0402_1005Metric, F.Cu at (146.2, 122.9)
- added C41: 100nF, Capacitor_SMD:C_0402_1005Metric, F.Cu at (146.2, 124.9)
- added C42: 100nF, Capacitor_SMD:C_0402_1005Metric, F.Cu at (146.2, 126.8)
- added L5: 345uH, custom_footprints:Generic_Solder_Pads_2P, F.Cu at (147.1, 95.7)
- added L6: JYLRA0832Z, custom_footprints:Generic_Solder_Pads_2P, F.Cu at (150.2, 121.5)
- added R41: 10k, Resistor_SMD:R_0402_1005Metric, F.Cu at (144.6, 102.0)
- added R42: 100k, Resistor_SMD:R_0402_1005Metric, F.Cu at (144.6, 103.9)
- added R43: 1k, Resistor_SMD:R_0603_1608Metric, F.Cu at (139.3, 105.6)
- added R44: 47k, Resistor_SMD:R_0402_1005Metric, F.Cu at (144.6, 105.9)
- added R47: 100k, Resistor_SMD:R_0402_1005Metric, F.Cu at (160.2, 104.8)
- added R49: 7.5k, Resistor_SMD:R_0603_1608Metric, F.Cu at (160.7, 102.6)
- added TP10: SCL, TestPoint:TestPoint_Pad_D1.0mm, F.Cu at (153.1, 95.7)
- added TP11: SDA, TestPoint:TestPoint_Pad_D1.0mm, F.Cu at (153.1, 98.7)
- added TP12: UART2_TX, TestPoint:TestPoint_Pad_D1.0mm, F.Cu at (153.1, 101.8)
- added TP13: UART2_RX, TestPoint:TestPoint_Pad_D1.0mm, F.Cu at (161.5, 155.0)
- added U11: SN74AUP1G17, Package_TO_SOT_SMD:Diodes_SOT-553, F.Cu at (146.4, 99.1)
- added U12: MKDV1GCL-ABA, MKDV1GCL-ABA:LGA-8_L6.0-W8.0-P1.27-TL, F.Cu at (157.3, 160.1)
- added U13: ST25R3916B-AQET, ST25R3916B-AQET:QFN-32_L5.0-W5.0-P0.50-TL-EP3.5, F.Cu at (175.0, 158.5)
- added U14: DRV2603RUNT, DRV2603RUNT:QFN-10_L2.0-W2.0-P0.50-TL, F.Cu at (153.2, 124.8)
- added U6: LIS2DW12TR, LIS2DW12TR:LGA-12_L2.0-W2.0-P0.50-BL, F.Cu at (149.4, 124.7)
- added Y3: 32.768khz, Crystal:Crystal_SMD_2012-2Pin_2.0x1.2mm, F.Cu at (156.7, 102.9)
- J1: value USB4215-03-A_REVA -> TYPE-C 16PIN 2MD(073); footprint USB4215-03-A:GCT_USB4215-03-A_REVA -> TYPE-C-16PIN-2MD-073:USB-C-SMD_TYPE-C-6PIN-2MD-073
- TP8: value SCL_G1 -> SCL_G2; footprint TestPoint:TestPoint_Pad_1.5x1.5mm -> TestPoint:TestPoint_Pad_D1.0mm
- TP9: value SDA_G1 -> SDA_G2; footprint TestPoint:TestPoint_Pad_1.5x1.5mm -> TestPoint:TestPoint_Pad_D1.0mm
- U4, U5: value USBLC6-2SC6 -> USBLC6-2P6; footprint Package_TO_SOT_SMD:SOT-23-6 -> Package_TO_SOT_SMD:SOT-666
- U7, U8: value MTCH2120-V/REB -> CAP1208-1-A4-TR; footprint MTCH2120:QFN_MTCH2120-V&slash_REB_MCH -> CAP1208-1-A4-TR:QFN16_3x3MC_MCH
- moved U4 53.0 mm to (157.6, 110.8), turned to 0 degrees
- moved U5 43.5 mm to (157.6, 114.2), turned to 0 degrees
- moved D3 37.8 mm to (140.2, 102.6)
- moved U8 33.1 mm to (143.1, 155.8)
- moved U7 26.7 mm to (149.9, 150.8)
- moved R3 12.8 mm to (158.4, 124.0)
- moved J1 1.44 mm to (124.9, 151.5)
Connections:
- C24 pad 1: +3V3 -> +3V3_G1
- D3 pad 1: RF_WAKE -> Net-(D3-K)
- Q1 pad 1: RF_MOD -> RF_DAT
- R3 pad 2: Net-(U2-GPOUT) -> FUEL_GPOUT
- TP8 pad 1: SCL_G1 -> SCL_G2
- TP9 pad 1: SDA_G1 -> SDA_G2
- U1 pad 1: SDA_G1 -> SDA_T1
- U1 pad 2: unconnected-(U1B-PA31-Pad2) -> SCL_T2
- U1 pad 25: HAPTIC_PWM -> FUEL_GPOUT
- U1 pad 28: FLASH_DIO3 -> SD_DAT1
- U1 pad 29: FLASH_CLK -> SD_DAT0
- U1 pad 3: unconnected-(U1B-PA30-Pad3) -> SDA_T2
- U1 pad 30: FLASH_DIO0 -> SD_CMD
- U1 pad 31: FLASH_DIO2 -> SD_CLK
- U1 pad 32: FLASH_DIO1 -> SD_DAT3
- U1 pad 33: FLASH_CS -> SD_DAT2
- U1 pad 35: unconnected-(U1B-PA10-Pad35) -> UART2_RX
- U1 pad 4: unconnected-(U1B-PA29-Pad4) -> HAPTIC_PWM
- U1 pad 42: unconnected-(U1B-PA9-Pad42) -> UART2_TX
- U1 pad 5: unconnected-(U1B-PA28-Pad5) -> LED_EN
- U1 pad 56: TOUCH_RST -> NFC_INT
- U1 pad 57: TOUCH_INT -> ACC_INT
- U1 pad 58: unconnected-(U1B-PA42-Pad58) -> SCL
- U1 pad 59: SCL -> SDA
- U1 pad 6: LED_EN -> TOUCH_INT
- U1 pad 60: SDA -> NFC_CS
- U1 pad 61: unconnected-(U1B-PA39-Pad61) -> NFC_CLK
- U1 pad 62: unconnected-(U1B-PA38-Pad62) -> NFC_DI
- U1 pad 63: unconnected-(U1B-PA37-Pad63) -> NFC_DO
- U1 pad 67: SCL_G1 -> SCL_T1
- U1 pad 7: unconnected-(U1B-PA26-Pad7) -> RF_WAKE
- U1 pad 8: unconnected-(U1B-PA25-Pad8) -> RF_DAT
- U2 pad A1: Net-(U2-GPOUT) -> FUEL_GPOUT
- U7 pad 1: SCL_G1 -> TOUCH_INT
- U7 pad 10: Net-(U7-BUTTON5/GPIO5) -> unconnected-(U7-CS7-Pad10)
- U7 pad 11: TOUCH_INT -> unconnected-(U7-CS6-Pad11)
- U7 pad 12: GND -> unconnected-(U7-CS5-Pad12)
- U7 pad 13: Net-(U7-BUTTON6/GPIO6) -> unconnected-(U7-CS4-Pad13)
- U7 pad 14: Net-(U7-BUTTON7/GPIO7) -> unconnected-(U7-CS3-Pad14)
- U7 pad 15: Net-(U7-BUTTON8/GPIO8) -> unconnected-(U7-CS2-Pad15)
- U7 pad 16: Net-(U7-BUTTON9/GPIO9) -> unconnected-(U7-CS1-Pad16)
- U7 pad 17: Net-(U7-BUTTON10/GPIO10) -> GND
- U7 pad 2: GND -> SDA_T1
- U7 pad 3: GND -> SCL_T1
- U7 pad 4: +3V3_G1 -> +3V3_G2
- U7 pad 5: Net-(U7-BUTTON0/GPIO0) -> unconnected-(U7-NC-Pad5)
- U7 pad 6: Net-(U7-BUTTON1/GPIO1) -> unconnected-(U7-NC-Pad6)
- U7 pad 7: Net-(U7-BUTTON2/GPIO2) -> GND
- U7 pad 8: Net-(U7-BUTTON3/GPIO3) -> GND
- U7 pad 9: Net-(U7-BUTTON4/GPIO4) -> unconnected-(U7-CS8-Pad9)
- U8 pad 1: SCL_G1 -> TOUCH_INT
- U8 pad 10: Net-(U8-BUTTON5/GPIO5) -> unconnected-(U8-CS7-Pad10)
- U8 pad 11: TOUCH_INT -> unconnected-(U8-CS6-Pad11)
- U8 pad 12: GND -> unconnected-(U8-CS5-Pad12)
- U8 pad 13: Net-(U8-BUTTON6/GPIO6) -> unconnected-(U8-CS4-Pad13)
- U8 pad 14: Net-(U8-BUTTON7/GPIO7) -> unconnected-(U8-CS3-Pad14)
- U8 pad 15: Net-(U8-BUTTON8/GPIO8) -> unconnected-(U8-CS2-Pad15)
- U8 pad 16: Net-(U8-BUTTON9/GPIO9) -> unconnected-(U8-CS1-Pad16)
- U8 pad 17: Net-(U8-BUTTON10/GPIO10) -> GND
- U8 pad 2: +3V3_G1 -> SDA_T2
- U8 pad 3: GND -> SCL_T2
- U8 pad 4: +3V3_G1 -> +3V3_G2
- U8 pad 5: Net-(U8-BUTTON0/GPIO0) -> unconnected-(U8-NC-Pad5)
- U8 pad 6: Net-(U8-BUTTON1/GPIO1) -> unconnected-(U8-NC-Pad6)
- U8 pad 7: Net-(U8-BUTTON2/GPIO2) -> GND
- U8 pad 8: Net-(U8-BUTTON3/GPIO3) -> GND
- U8 pad 9: Net-(U8-BUTTON4/GPIO4) -> unconnected-(U8-CS8-Pad9)

Commit message: push changes before removing fuel gauge
Parts:
- removed J2: U.FL-R-SMT-1(10), U.FL-R-SMT-1_10_:HRS_U.FL-R-SMT-1_10_
- moved R41 14.8 mm to (135.9, 114.0)
- moved R42 14.8 mm to (135.9, 116.0)
- moved R44 14.8 mm to (135.9, 118.0)
- moved C34 14.8 mm to (138.8, 114.0)
- moved L5 14.8 mm to (138.4, 107.8)
- moved R43 14.8 mm to (130.7, 117.6)
- moved TP11 14.8 mm to (144.5, 110.8)
- moved TP12 14.8 mm to (144.5, 113.8)
- moved U11 14.8 mm to (137.8, 111.2)
- moved Y3 14.8 mm to (148.1, 115.0)
- moved D3 14.8 mm to (131.6, 114.7)
- moved R47 14.8 mm to (151.5, 116.9)
- moved R49 14.8 mm to (152.1, 114.6)
- moved TP10 14.8 mm to (144.5, 107.7)
- moved LED1 0.43 mm to (136.5, 162.8)
