File: rc_keychain.kicad_pcb (KiCad board)
At the start: 2 copper layers, 58 x 18 mm, 102 parts, among them J1 TYPE-C 16PIN 2MD(073), J5 5034801200, Q1 2N7002, SW2 TS35CA, U1 SF32LB525UC6, U10 TPS61040DBV, U11 SN74AUP1G17, U12 MKDV1GCL-ABA, U13 ST25R3916B-AQET, U14 DRV2603RUNT, U2 BQ27426YZFR, U3 TPS25200DRVT, U4 USBLC6-2P6, U5 USBLC6-2P6, U6 LIS2DW12TR, U7 CAP1208-1-A4-TR, U8 CAP1208-1-A4-TR, U9 AP3602AKTR-G1, Y2 48MHz, Y3 32.768khz

Commit message: hopefully final schematic before splitting out
Parts:
- removed J1: TYPE-C 16PIN 2MD(073), TYPE-C-16PIN-2MD-073:USB-C-SMD_TYPE-C-6PIN-2MD-073
- removed R37, R42, R47: 100k, Resistor_SMD:R_0402_1005Metric
- removed R38: 560k, Resistor_SMD:R_0402_1005Metric
- removed R39: 820k, Resistor_SMD:R_0402_1005Metric
- removed R40: 130k, Resistor_SMD:R_0402_1005Metric
- removed R41: 10k, Resistor_SMD:R_0402_1005Metric
- removed R43: 1k, Resistor_SMD:R_0603_1608Metric
- removed R44: 47k, Resistor_SMD:R_0402_1005Metric
- removed R49: 7.5k, Resistor_SMD:R_0603_1608Metric
- removed SW2: TS35CA, TS35CA:KEY-SMD_TS35CA
- removed U14: DRV2603RUNT, DRV2603RUNT:QFN-10_L2.0-W2.0-P0.50-TL
- added C35: 100nF, Capacitor_SMD:C_0402_1005Metric, F.Cu at (148.5, 81.8)
- added C36: 1uF, Capacitor_SMD:C_0402_1005Metric, F.Cu at (148.5, 83.8)
- added C37: 10uF, Capacitor_SMD:C_0402_1005Metric, F.Cu at (148.5, 85.7)
- added C38: 4.7nF, Capacitor_SMD:C_0402_1005Metric, F.Cu at (177.5, 71.3)
- added C43: 22nF, Capacitor_SMD:C_0402_1005Metric, F.Cu at (195.6, 109.2)
- added C44: 10nF, Capacitor_SMD:C_0402_1005Metric, F.Cu at (195.6, 111.1)
- added C45: 10nF, Capacitor_SMD:C_0402_1005Metric, F.Cu at (196.0, 97.2)
- added C46: 2.2uF, Capacitor_SMD:C_0402_1005Metric, F.Cu at (196.0, 99.2)
- added C47: 2.2uF, Capacitor_SMD:C_0402_1005Metric, F.Cu at (198.3, 96.2)
- added C48: 10nF, Capacitor_SMD:C_0402_1005Metric, F.Cu at (198.3, 98.2)
- added C49: 2.2uF, Capacitor_SMD:C_0402_1005Metric, F.Cu at (197.8, 107.2)
- added C50: 10nF, Capacitor_SMD:C_0402_1005Metric, F.Cu at (197.8, 109.2)
- added C51: 2.2uF, Capacitor_SMD:C_0402_1005Metric, F.Cu at (197.8, 111.1)
- added C52: 10nF, Capacitor_SMD:C_0402_1005Metric, F.Cu at (197.8, 108.2)
- added C53: 2.2uF, Capacitor_SMD:C_0402_1005Metric, F.Cu at (198.2, 97.2)
- added C54: 10nF, Capacitor_SMD:C_0402_1005Metric, F.Cu at (200.5, 96.2)
- added C55: 1uF, Capacitor_SMD:C_0402_1005Metric, F.Cu at (200.5, 98.0)
- added C56: 10nF, Capacitor_SMD:C_0402_1005Metric, F.Cu at (200.5, 107.2)
- added C57: 680pF, Capacitor_SMD:C_0402_1005Metric, F.Cu at (200.5, 109.2)
- added C58: 58pF, Capacitor_SMD:C_0402_1005Metric, F.Cu at (200.5, 111.1)
- added C59: 3pF, Capacitor_SMD:C_0402_1005Metric, F.Cu at (200.8, 99.2)
- added C60: 10pF, Capacitor_SMD:C_0402_1005Metric, F.Cu at (198.2, 99.2)
- added C61: 220pF, Capacitor_SMD:C_0402_1005Metric, F.Cu at (195.7, 108.2)
- added J2: TYPE-C 16PIN 2MD(073), TYPE-C-16PIN-2MD-073:USB-C-SMD_TYPE-C-6PIN-2MD-073, F.Cu at (147.8, 100.2)
- added J3: Touch_Surface_Top, custom_footprints:Touch_Surface_8_Pad, F.Cu at (182.2, 113.2)
- added J4: Touch_Surface_Bottom, custom_footprints:Touch_Surface_8_Pad, F.Cu at (182.2, 93.8)
- added L7: 1462360151, custom_footprints:Generic_Solder_Pads_2P, F.Cu at (192.0, 96.2)
- added L8: 270nH, Inductor_SMD:L_0603_1608Metric, F.Cu at (193.5, 103.3)
- added R10: 4.7k, Resistor_SMD:R_0402_1005Metric, F.Cu at (180.1, 78.8)
- added R13: 4.7k, Resistor_SMD:R_0402_1005Metric, F.Cu at (180.1, 84.8)
- added R14: 560k, Resistor_SMD:R_0402_1005Metric, F.Cu at (151.4, 77.9)
- added R15: 130k, Resistor_SMD:R_0402_1005Metric, F.Cu at (151.4, 79.8)
- added R16: 820k, Resistor_SMD:R_0402_1005Metric, F.Cu at (151.4, 81.8)
- added R17: 5.1k, Resistor_SMD:R_0402_1005Metric, F.Cu at (151.4, 83.8)
- added R18: 10k, Resistor_SMD:R_0402_1005Metric, F.Cu at (151.4, 85.8)
- added R19: 100k, Resistor_SMD:R_0402_1005Metric, F.Cu at (151.4, 87.8)
- added R20: 10k, Resistor_SMD:R_0402_1005Metric, F.Cu at (189.0, 77.5)
- added R21: 47k, Resistor_SMD:R_0402_1005Metric, F.Cu at (189.0, 79.5)
- added R22: 100k, Resistor_SMD:R_0402_1005Metric, F.Cu at (189.0, 81.5)
- added R23: 1k, Resistor_SMD:R_0603_1608Metric, F.Cu at (194.6, 74.1)
- added R24: 5.8, Resistor_SMD:R_0402_1005Metric, F.Cu at (193.7, 98.0)
- added R8: 5.1k, Resistor_SMD:R_0402_1005Metric, F.Cu at (188.3, 86.7)
- added R9: 5.1k, Resistor_SMD:R_0402_1005Metric, F.Cu at (188.3, 88.7)
- added SW1: TS35CA, TS35CA:KEY-SMD_TS35CA, F.Cu at (154.2, 111.0)
- added TP14: NFC_CSO, TestPoint:TestPoint_Pad_D1.0mm, F.Cu at (207.7, 107.0)
- added TP15: NFC_CSI, TestPoint:TestPoint_Pad_D1.0mm, F.Cu at (210.2, 112.0)
- added Y1: 48MHz, Crystal:Crystal_SMD_2520-4Pin_2.5x2.0mm, F.Cu at (160.8, 65.6)
- C1: value 4.7uF -> NF
- C10: value 470nF -> 4.7uF; footprint Capacitor_SMD:C_0603_1608Metric -> Capacitor_SMD:C_0402_1005Metric
- C11: value 4.7uF -> 2.2uF
- C12: value 4.7uF -> 1uF
- C13, C27: value 1uF -> 4.7uF
- C14: value 2.2uF -> 4.7uF
- C15: value 4.7uF -> 470nF; footprint Capacitor_SMD:C_0402_1005Metric -> Capacitor_SMD:C_0603_1608Metric
- C16: value 4.7uF -> 10uF
- C17, C19: value 10uF -> 4.7uF
- C2: value 470nF -> 15pF; footprint Capacitor_SMD:C_0603_1608Metric -> Capacitor_SMD:C_0402_1005Metric
- C20: value NF -> 10uF; footprint Capacitor_SMD:C_0603_1608Metric -> Capacitor_SMD:C_0402_1005Metric
- C21: value 15pF -> 4.7uF
- C22, C23: value NF -> 100nF
- C24, C25: value 100nF -> 1uF
- C26: value 10uF -> 100nF
- C28: value 10uF -> 2.2uF; footprint Capacitor_SMD:C_0402_1005Metric -> Capacitor_SMD:C_0603_1608Metric
- C29: value 2.2uF -> 15pF; footprint Capacitor_SMD:C_0603_1608Metric -> Capacitor_SMD:C_0402_1005Metric
- C3: value 2.2uF -> NF
- C30: footprint Capacitor_SMD:C_0402_1005Metric -> Capacitor_SMD:C_0603_1608Metric
- C31: value 15pF -> 100nF
- C32: value 4.7uF -> 10uF; footprint Capacitor_SMD:C_0603_1608Metric -> Capacitor_SMD:C_0402_1005Metric
- C33: value 4.7nF -> 100nF
- C34: value 10nF -> 10uF
- C39: value 100nF -> 10nF
- C4: value 4.7uF -> NF; footprint Capacitor_SMD:C_0402_1005Metric -> Capacitor_SMD:C_0603_1608Metric
- C40: value 10uF -> 10pF
- C41: value 100nF -> 10pF
- C42: value 100nF -> 2.2uF
- C6: value 22uF -> 100nF; footprint Capacitor_SMD:C_0603_1608Metric -> Capacitor_SMD:C_0402_1005Metric
- C7: value 10uF -> 22uF; footprint Capacitor_SMD:C_0402_1005Metric -> Capacitor_SMD:C_0603_1608Metric
- C9: value 1uF -> 10uF
- L1: value 4.7uH -> NF; footprint Inductor_SMD:L_0402_1005Metric -> Inductor_SMD:L_0603_1608Metric
- L3: value NF -> 4.7uH; footprint Inductor_SMD:L_0603_1608Metric -> Inductor_SMD:L_0402_1005Metric
- L5: value 345uH -> JYLRA0832Z
- L6: value JYLRA0832Z -> 345uH
- R1: value 10k -> 7.5k; footprint Resistor_SMD:R_0402_1005Metric -> Resistor_SMD:R_0603_1608Metric
- R11: value 5.1k -> 4.7k
- R12: value 10k -> 4.7k
- R2: value 0.01 -> 4.7k; footprint Resistor_SMD:R_1206_3216Metric -> Resistor_SMD:R_0402_1005Metric
- R3: value 10k -> 100k
- R4: value 300k -> 4.7k; footprint Resistor_SMD:R_0603_1608Metric -> Resistor_SMD:R_0402_1005Metric
- R5: value 150k -> 300k
- R7: value 5.1k -> 150k; footprint Resistor_SMD:R_0402_1005Metric -> Resistor_SMD:R_0603_1608Metric
- TP1: value DBG_A -> UART2_TX
- TP10: value SCL -> GND
- TP11: value SDA -> 3V3
- TP12: value UART2_TX -> USB_DP
- TP13: value UART2_RX -> USB_DM
- TP2: value DBG_B -> UART2_RX
- TP3: value VBAT -> DBG_A
- TP4: value GND -> DBG_B
- TP5: value 3V3 -> SDA
- TP6: value USB_DP -> SCL
- TP7: value USB_DM -> SCL_G2
- TP8: value SCL_G2 -> SDA_G2
- TP9: value SDA_G2 -> VBAT
- U10: value TPS61040DBV -> LIS2DW12TR; footprint Package_TO_SOT_SMD:SOT-23-5 -> LIS2DW12TR:LGA-12_L2.0-W2.0-P0.50-BL
- U11: value SN74AUP1G17 -> AP3602AKTR-G1; footprint Package_TO_SOT_SMD:Diodes_SOT-553 -> AP3602AKTR-G1:SOT-23-6_L2.9-W1.6-P0.95-LS2.8-BR
- U12: value MKDV1GCL-ABA -> SN74AUP1G17; footprint MKDV1GCL-ABA:LGA-8_L6.0-W8.0-P1.27-TL -> Package_TO_SOT_SMD:Diodes_SOT-553
- U2: value BQ27426YZFR -> MKDV1GCL-ABA; footprint BQ27426:YZF0009AKAL -> MKDV1GCL-ABA:LGA-8_L6.0-W8.0-P1.27-TL
- U6: value LIS2DW12TR -> CAP1208-1-A4-TR; footprint LIS2DW12TR:LGA-12_L2.0-W2.0-P0.50-BL -> CAP1208-1-A4-TR:QFN16_3x3MC_MCH
- U8: value CAP1208-1-A4-TR -> DRV2603RUNT; footprint CAP1208-1-A4-TR:QFN16_3x3MC_MCH -> DRV2603RUNT:QFN-10_L2.0-W2.0-P0.50-TL
- U9: value AP3602AKTR-G1 -> TPS61040DBV; footprint AP3602AKTR-G1:SOT-23-6_L2.9-W1.6-P0.95-LS2.8-BR -> Package_TO_SOT_SMD:SOT-23-5
- Y2: value 48MHz -> 32.768khz; footprint Crystal:Crystal_SMD_2520-4Pin_2.5x2.0mm -> Crystal:Crystal_SMD_2012-2Pin_2.0x1.2mm
- Y3: value 32.768khz -> 27.12MHz; footprint Crystal:Crystal_SMD_2012-2Pin_2.0x1.2mm -> Crystal:Crystal_SMD_2016-4Pin_2.0x1.6mm
- moved U12 96.0 mm to (177.5, 66.3)
- moved LED1 94.6 mm to (158.4, 70.7)
- moved TP2 89.3 mm to (213.7, 116.5)
- moved TP1 89.3 mm to (213.7, 113.5)
- moved U10 88.0 mm to (162.7, 74.6)
- moved TP8 87.9 mm to (222.8, 116.5)
- moved TP9 87.1 mm to (217.0, 104.4)
- moved TP6 85.9 mm to (219.8, 116.5)
- moved U9 82.6 mm to (162.0, 79.3)
- moved U3 80.1 mm to (177.8, 88.3)
- moved R2 79.0 mm to (172.6, 71.3), turned to 0 degrees
- moved D1 76.1 mm to (160.5, 83.4)
- moved Y2 76.1 mm to (153.3, 73.0)
- moved C4 75.7 mm to (149.3, 64.8)
- moved TP7 74.7 mm to (222.8, 113.5)
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Connections:
- BT1 pad 1: Net-(BT1-+) -> VBAT
- C1 pad 1: VBAT -> Net-(U1B-ANT)
- C10 pad 1: Net-(U1A-VDD_RET) -> Net-(U1A-GPADC_VREF)
- C11 pad 1: Net-(U1A-VDD_VOUT2) -> Net-(U1A-VDD18_VOUT)
- C12 pad 1: Net-(U1A-VDD_VOUT1) -> Net-(U1A-VDD_RTC)
- C13 pad 1: Net-(U1A-VDD_RTC) -> Net-(U1A-VDD_VOUT1)
- C14 pad 1: Net-(U1A-VDD18_VOUT) -> Net-(U1A-VDD_VOUT2)
- C15 pad 1: Net-(U1A-GPADC_VREF) -> Net-(U1A-VDD_RET)
- C16 pad 1: +3V3 -> +3V3_G2
- C17 pad 1: +3V3 -> VBAT
- C18 pad 1: +3V3_G2 -> +3V3
- C19 pad 1: +3V3_G1 -> +3V3
- C2 pad 1: Net-(U2-VDD) -> Net-(U1B-ANT)
- C2 pad 2: GND -> Net-(C2-Pad2)
- C20 pad 1: Net-(C20-Pad1) -> +3V3_G1
- C20 pad 2: Net-(C20-Pad2) -> GND
- C21 pad 1: Net-(U1B-ANT) -> Net-(U1A-BUCK_FB)
- C21 pad 2: Net-(C20-Pad1) -> GND
- C22 pad 1: Net-(U1B-ANT) -> +3V3_G2
- C23 pad 1: Net-(C20-Pad1) -> +3V3_G2
- C24 pad 1: +3V3_G1 -> +3V3_G2
- C25 pad 1: BUTTON -> +3V3_G2
- C27 pad 1: Net-(U9-C+) -> VBAT
- C27 pad 2: Net-(U9-C-) -> GND
- C28 pad 1: +5V -> GND
- C28 pad 2: GND -> Net-(J5-VCOMH)
- C29 pad 1: GND -> +9V
- C29 pad 2: Net-(J5-VCOMH) -> Net-(U9-FB)
- C3 pad 1: Net-(U2-VDD) -> Net-(C2-Pad2)
- C30 pad 1: VBAT -> +9V
- C31 pad 1: +9V -> BUTTON
- C31 pad 2: Net-(U10-FB) -> GND
- C32 pad 1: +9V -> VBAT
- C33 pad 1: Net-(D2-K) -> +3V3
- C34 pad 1: GND -> +3V3
- C34 pad 2: Net-(D2-A) -> GND
- C39 pad 1: +3V3 -> GND
- C39 pad 2: GND -> Net-(D2-A)
- C4 pad 1: Net-(U1A-BUCK_FB) -> Net-(C2-Pad2)
- C4 pad 2: GND -> Net-(C4-Pad2)
- C40 pad 1: +3V3 -> /rf/XTI
- C41 pad 1: +3V3 -> /rf/XTO
- C42 pad 1: VBAT -> /rf/VDD_AM
- C5 pad 1: VBUS_RAW -> +3V3_G1
- C6 pad 1: VBUS -> VBUS_RAW
- C7 pad 1: VBAT -> VBUS
- C9 pad 1: Net-(BT1-+) -> VBAT
- L1 pad 1: Net-(U1A-BUCK_LX) -> Net-(C4-Pad2)
- L1 pad 2: Net-(U1A-BUCK_FB) -> GND
- L2 pad 1: Net-(C20-Pad2) -> Net-(C4-Pad2)
- L3 pad 1: Net-(C20-Pad2) -> Net-(U1A-BUCK_LX)
- L3 pad 2: GND -> Net-(U1A-BUCK_FB)
- L5 pad 1: GND -> /interface/LRA_OUTP
- L5 pad 2: Net-(D2-K) -> /interface/LRA_OUTN
- L6 pad 1: /interface/LRA_OUTP -> GND
- L6 pad 2: /interface/LRA_OUTN -> Net-(D2-K)
- R1 pad 1: Net-(U2-BIN) -> +3V3_G1
- R1 pad 2: GND -> SD_DAT3
- R11 pad 1: +3V3 -> +3V3_G2
- R11 pad 2: Net-(R11-Pad2) -> SDA_T2
- R12 pad 1: BUTTON -> +3V3_G2
- R12 pad 2: GND -> SCL_T1
- R2 pad 1: Net-(BT1-+) -> +3V3
- R2 pad 2: VBAT -> SDA
- R3 pad 1: +3V3 -> TOUCH_INT
- R3 pad 2: FUEL_GPOUT -> +3V3_G2
- R4 pad 1: VBUS_RAW -> +3V3
- R4 pad 2: Net-(U3-EN) -> SCL
- R5 pad 1: Net-(U3-ILIM) -> VBUS_RAW
- R5 pad 2: GND -> Net-(U3-EN)
- R7 pad 1: Net-(J1-CC1) -> Net-(U3-ILIM)
- TP1 pad 1: DBG_A -> UART2_TX
- TP10 pad 1: SCL -> GND
- TP11 pad 1: SDA -> +3V3
- TP12 pad 1: UART2_TX -> USB_DP
- TP13 pad 1: UART2_RX -> USB_DM
- TP2 pad 1: DBG_B -> UART2_RX
- TP3 pad 1: Net-(BT1-+) -> DBG_A
- TP4 pad 1: GND -> DBG_B
- TP5 pad 1: +3V3 -> SDA
- TP6 pad 1: USB_DP -> SCL
- TP7 pad 1: USB_DM -> SCL_G2
- TP8 pad 1: SCL_G2 -> SDA_G2
- TP9 pad 1: SDA_G2 -> VBAT
- U10 pad 1: Net-(D1-K) -> SCL
- U10 pad 2: GND -> unconnected-(U10-CS-Pad2)
- U10 pad 3: Net-(U10-FB) -> unconnected-(U10-SDO/SA0-Pad3)
- U10 pad 4: OLED_EN -> SDA
- U10 pad 5: VBAT -> GND
- U11 pad 1: unconnected-(U11-NC-Pad1) -> +5V
- U11 pad 2: Net-(D3-K) -> GND
- U11 pad 3: GND -> LED_EN
- U11 pad 4: RF_WAKE -> Net-(U11-C-)
- U11 pad 5: +3V3 -> VBAT
- U12 pad 1: SD_DAT2 -> unconnected-(U12-NC-Pad1)
- U12 pad 2: SD_DAT3 -> Net-(D3-K)
- U12 pad 3: SD_CLK -> GND
- U12 pad 4: GND -> RF_WAKE
- U12 pad 5: SD_CMD -> +3V3
- U13 pad 10: unconnected-(U13-VDD_TX-Pad10) -> +3V3
- U13 pad 11: unconnected-(U13-VDD_AM-Pad11) -> /rf/VDD_AM
- U13 pad 13: unconnected-(U13-RFO1-Pad13) -> /rf/RFO1
- U13 pad 14: unconnected-(U13-VDD_DR-Pad14) -> /rf/VDD_RF
- U13 pad 2: unconnected-(U13-CSO-Pad2) -> Net-(U13-CSO)
- U13 pad 20: unconnected-(U13-I2C_EN-Pad20) -> GND
- U13 pad 21: unconnected-(U13-VSS-Pad21) -> GND
- U13 pad 22: unconnected-(U13-RFI1-Pad22) -> /rf/RFI1
- U13 pad 24: unconnected-(U13-AGDC-Pad24) -> Net-(U13-AGDC)
- U13 pad 25: unconnected-(U13-CSI-Pad25) -> Net-(U13-CSI)
- U13 pad 26: unconnected-(U13-GND_A-Pad26) -> GND
- U13 pad 27: unconnected-(U13-IRQ-Pad27) -> NFC_INT
- U13 pad 3: unconnected-(U13-VDD_D-Pad3) -> /rf/VDD_D
- U13 pad 33: unconnected-(U13-EP-Pad33) -> GND
- U13 pad 4: unconnected-(U13-XTO-Pad4) -> /rf/XTO
- U13 pad 5: unconnected-(U13-XTI-Pad5) -> /rf/XTI
- U13 pad 6: unconnected-(U13-GND_D-Pad6) -> GND
- U13 pad 7: unconnected-(U13-VDD_A-Pad7) -> /rf/VDD_A
- U13 pad 8: unconnected-(U13-VDD-Pad8) -> +3V3
- U13 pad 9: unconnected-(U13-VDD_RF-Pad9) -> /rf/VDD_RF
- U6 pad 1: SCL -> TOUCH_INT
- U6 pad 10: +3V3 -> Net-(J3-Pin_7)
- U6 pad 11: unconnected-(U6-INT2-Pad11) -> Net-(J3-Pin_6)
- U6 pad 12: ACC_INT -> Net-(J3-Pin_5)
- U6 pad 2: unconnected-(U6-CS-Pad2) -> SDA_T1
- U6 pad 3: unconnected-(U6-SDO/SA0-Pad3) -> SCL_T1
- U6 pad 4: SDA -> +3V3_G2
- U6 pad 5: GND -> unconnected-(U6-NC-Pad5)
- U6 pad 6: GND -> unconnected-(U6-NC-Pad6)
- U6 pad 9: +3V3 -> Net-(J3-Pin_8)
- U7 pad 10: unconnected-(U7-CS7-Pad10) -> Net-(J4-Pin_7)
- U7 pad 11: unconnected-(U7-CS6-Pad11) -> Net-(J4-Pin_6)
- U7 pad 12: unconnected-(U7-CS5-Pad12) -> Net-(J4-Pin_5)
- U7 pad 13: unconnected-(U7-CS4-Pad13) -> Net-(J4-Pin_4)
- U7 pad 14: unconnected-(U7-CS3-Pad14) -> Net-(J4-Pin_3)
- U7 pad 15: unconnected-(U7-CS2-Pad15) -> Net-(J4-Pin_2)
- U7 pad 16: unconnected-(U7-CS1-Pad16) -> Net-(J4-Pin_1)
- U7 pad 2: SDA_T1 -> SDA_T2
- U7 pad 3: SCL_T1 -> SCL_T2
- U7 pad 9: unconnected-(U7-CS8-Pad9) -> Net-(J4-Pin_8)
- U8 pad 1: TOUCH_INT -> +3V3
- U8 pad 10: unconnected-(U8-CS7-Pad10) -> GND
- U8 pad 2: SDA_T2 -> HAPTIC_PWM
- U8 pad 3: SCL_T2 -> +3V3
- U8 pad 4: +3V3_G2 -> unconnected-(U8-NC-Pad4)
- U8 pad 5: unconnected-(U8-NC-Pad5) -> GND
- U8 pad 6: unconnected-(U8-NC-Pad6) -> /interface/LRA_OUTN
- U8 pad 7: GND -> VBAT
- U8 pad 9: unconnected-(U8-CS8-Pad9) -> /interface/LRA_OUTP
- U9 pad 1: +5V -> Net-(D1-K)
- U9 pad 3: LED_EN -> Net-(U9-FB)
- U9 pad 4: Net-(U9-C-) -> OLED_EN
- Y2 pad 1: Net-(U1B-XTAL48M_XO) -> Net-(U1B-PA23)
- Y2 pad 2: GND -> Net-(U1B-PA22)
- Y3 pad 1: Net-(U1B-PA23) -> /rf/XTI
- Y3 pad 2: Net-(U1B-PA22) -> GND

Commit message: huge progress on bentoboard, schematic fixes
Parts:
- added D4: ESD5341N, Diode_SMD:D_SOD-882, F.Cu at (105.7, 66.0)
- added J1: U.FL-R-SMT-1(10), U.FL-R-SMT-1_10_:HRS_U.FL-R-SMT-1_10_, F.Cu at (110.6, 134.8)
- added JP1: USB_OVP_FAULT, Jumper:SolderJumper-2_P1.3mm_Open_Pad1.0x1.5mm, F.Cu at (122.4, 60.5)
- added JP10: OLED_DC, Jumper:SolderJumper-2_P1.3mm_Open_Pad1.0x1.5mm, F.Cu at (162.6, 91.7)
- added JP11: OLED_CLK, Jumper:SolderJumper-2_P1.3mm_Open_Pad1.0x1.5mm, F.Cu at (166.5, 91.7)
- added JP12: OLED_DAT, Jumper:SolderJumper-2_P1.3mm_Open_Pad1.0x1.5mm, F.Cu at (170.3, 91.7)
- added JP13: OLED_9V, Jumper:SolderJumper-2_P1.3mm_Open_Pad1.0x1.5mm, F.Cu at (179.4, 91.9)
- added JP14: ACC_SCL, Jumper:SolderJumper-2_P1.3mm_Open_Pad1.0x1.5mm, F.Cu at (126.5, 80.8)
- added JP15: ACC_SDA, Jumper:SolderJumper-2_P1.3mm_Open_Pad1.0x1.5mm, F.Cu at (126.5, 83.4)
- added JP16: ACC_3V3, Jumper:SolderJumper-2_P1.3mm_Open_Pad1.0x1.5mm, F.Cu at (126.5, 75.6)
- added JP17: ACC_INT, Jumper:SolderJumper-2_P1.3mm_Open_Pad1.0x1.5mm, F.Cu at (126.5, 78.2)
- added JP18: TOUCH_SCL_T1, Jumper:SolderJumper-2_P1.3mm_Open_Pad1.0x1.5mm, F.Cu at (145.0, 125.9)
- added JP19: TOUCH_SDA_T1, Jumper:SolderJumper-2_P1.3mm_Open_Pad1.0x1.5mm, F.Cu at (145.0, 123.3)
- added JP2: USB_VBUS, Jumper:SolderJumper-2_P1.3mm_Open_Pad1.0x1.5mm, F.Cu at (116.6, 68.7)
- added JP20: TOUCH_SCL_T2, Jumper:SolderJumper-2_P1.3mm_Open_Pad1.0x1.5mm, F.Cu at (145.0, 128.5)
- added JP21: TOUCH_SDA_T2, Jumper:SolderJumper-2_P1.3mm_Open_Pad1.0x1.5mm, F.Cu at (145.0, 131.1)
- added JP22: OLED_VBAT, Jumper:SolderJumper-2_P1.3mm_Open_Pad1.0x1.5mm, F.Cu at (174.2, 91.7)
- added JP23: TOUCH_3V3_G2, Jumper:SolderJumper-2_P1.3mm_Open_Pad1.0x1.5mm, F.Cu at (145.0, 133.7)
- added JP24: TOUCH_INT, Jumper:SolderJumper-2_P1.3mm_Open_Pad1.0x1.5mm, F.Cu at (145.0, 120.7)
- added JP26: HAPTIC_PWM, Jumper:SolderJumper-2_P1.3mm_Open_Pad1.0x1.5mm, F.Cu at (125.7, 87.8)
- added JP27: HAPTIC_EN, Jumper:SolderJumper-2_P1.3mm_Open_Pad1.0x1.5mm, F.Cu at (125.7, 90.5)
- added JP28: HAPTIC_VBAT, Jumper:SolderJumper-2_P1.3mm_Open_Pad1.0x1.5mm, F.Cu at (125.7, 93.0)
- added JP29: LED_EN, Jumper:SolderJumper-2_P1.3mm_Open_Pad1.0x1.5mm, F.Cu at (104.7, 117.3)
- added JP3: USB_DP, Jumper:SolderJumper-2_P1.3mm_Open_Pad1.0x1.5mm, F.Cu at (110.8, 68.7)
- added JP30: LED_DAT, Jumper:SolderJumper-2_P1.3mm_Open_Pad1.0x1.5mm, F.Cu at (103.5, 110.9)
- added JP31: LED_5V, Jumper:SolderJumper-2_P1.3mm_Open_Pad1.0x1.5mm, F.Cu at (98.2, 119.9)
- added JP32: LED_VBAT, Jumper:SolderJumper-2_P1.3mm_Open_Pad1.0x1.5mm, F.Cu at (103.5, 113.5)
- added JP33: RFID_DAT, Jumper:SolderJumper-2_P1.3mm_Open_Pad1.0x1.5mm, F.Cu at (133.8, 69.9)
- added JP34: RFID_WAKE, Jumper:SolderJumper-2_P1.3mm_Open_Pad1.0x1.5mm, F.Cu at (136.4, 69.9)
- added JP35: NFC_DI, Jumper:SolderJumper-2_P1.3mm_Open_Pad1.0x1.5mm, F.Cu at (149.3, 68.8)
- added JP36: NFC_DO, Jumper:SolderJumper-2_P1.3mm_Open_Pad1.0x1.5mm, F.Cu at (151.9, 68.8)
- added JP37: NFC_CLK, Jumper:SolderJumper-2_P1.3mm_Open_Pad1.0x1.5mm, F.Cu at (154.5, 68.8)
- added JP38: NFC_CS, Jumper:SolderJumper-2_P1.3mm_Open_Pad1.0x1.5mm, F.Cu at (157.1, 68.8)
- added JP39: NFC_INT, Jumper:SolderJumper-2_P1.3mm_Open_Pad1.0x1.5mm, F.Cu at (159.7, 68.8)
- added JP4: USB_DN, Jumper:SolderJumper-2_P1.3mm_Open_Pad1.0x1.5mm, F.Cu at (113.5, 68.7)
- added JP40: NFC_3V3, Jumper:SolderJumper-2_P1.3mm_Open_Pad1.0x1.5mm, F.Cu at (147.8, 80.5)
- added JP41: RFID_3V3, Jumper:SolderJumper-2_P1.3mm_Open_Pad1.0x1.5mm, F.Cu at (139.0, 69.9)
- added JP42: RFID_WAKE_RAW, Jumper:SolderJumper-2_P1.3mm_Open_Pad1.0x1.5mm, F.Cu at (132.7, 61.2)
- added JP43: OLED_EN, Jumper:SolderJumper-2_P1.3mm_Open_Pad1.0x1.5mm, F.Cu at (147.6, 91.6)
- added JP44: USB_3V3, Jumper:SolderJumper-2_P1.3mm_Open_Pad1.0x1.5mm, F.Cu at (119.5, 68.7)
- added JP5: USB_DBG_A, Jumper:SolderJumper-2_P1.3mm_Open_Pad1.0x1.5mm, F.Cu at (122.4, 63.1)
- added JP6: USB_DBG_B, Jumper:SolderJumper-2_P1.3mm_Open_Pad1.0x1.5mm, F.Cu at (122.4, 65.7)
- added JP7: OLED_3V3_G2, Jumper:SolderJumper-2_P1.3mm_Open_Pad1.0x1.5mm, F.Cu at (151.3, 91.6)
- added JP8: OLED_CS, Jumper:SolderJumper-2_P1.3mm_Open_Pad1.0x1.5mm, F.Cu at (155.1, 91.7)
- added JP9: OLED_RST, Jumper:SolderJumper-2_P1.3mm_Open_Pad1.0x1.5mm, F.Cu at (158.9, 91.7)
- added TP16: SCL_T2, TestPoint:TestPoint_Pad_D1.0mm, F.Cu at (133.0, 128.9)
- added TP17: SDA_T2, TestPoint:TestPoint_Pad_D1.0mm, F.Cu at (135.1, 127.4)
- added TP18: SD_CLK, TestPoint:TestPoint_Pad_D1.0mm, F.Cu at (121.1, 108.9)
- added TP19: SD_CLK, TestPoint:TestPoint_Pad_D1.0mm, F.Cu at (132.1, 115.9)
- added TP20: SD_DAT0, TestPoint:TestPoint_Pad_D1.0mm, F.Cu at (132.1, 113.8)
- added TP21: SD_DAT1, TestPoint:TestPoint_Pad_D1.0mm, F.Cu at (132.1, 111.7)
- added TP22: SD_DAT2, TestPoint:TestPoint_Pad_D1.0mm, F.Cu at (116.5, 115.1)
- added TP23: SD_DAT3, TestPoint:TestPoint_Pad_D1.0mm, F.Cu at (116.5, 113.0)
- added TP24: VBUS, TestPoint:TestPoint_Pad_D1.0mm, F.Cu at (119.4, 71.7)
- added TP25: DBG_C, TestPoint:TestPoint_Pad_D1.0mm, F.Cu at (120.8, 120.9)
- added TP26: 3V3_G1, TestPoint:TestPoint_Pad_D1.0mm, F.Cu at (131.2, 108.4)
- added TP27: 3V3_G2, TestPoint:TestPoint_Pad_D1.0mm, F.Cu at (135.0, 121.3)
- added TP28: 9V, TestPoint:TestPoint_Pad_D1.0mm, F.Cu at (179.0, 97.0)
- added TP29: OLED_CS, TestPoint:TestPoint_Pad_D1.0mm, F.Cu at (155.1, 87.5)
- added TP30: OLED_RST, TestPoint:TestPoint_Pad_D1.0mm, F.Cu at (158.9, 87.5)
- added TP31: OLED_DC, TestPoint:TestPoint_Pad_D1.0mm, F.Cu at (162.6, 87.5)
- added TP32: OLED_CLK, TestPoint:TestPoint_Pad_D1.0mm, F.Cu at (166.5, 87.5)
- added TP33: OLED_DAT, TestPoint:TestPoint_Pad_D1.0mm, F.Cu at (170.3, 87.5)
- added TP34: OLED_EN, TestPoint:TestPoint_Pad_D1.0mm, F.Cu at (147.6, 87.4)
- added TP35: HAPTIC_EN, TestPoint:TestPoint_Pad_D1.0mm, F.Cu at (132.2, 90.5)
- added TP36: HAPTIC_PWM, TestPoint:TestPoint_Pad_D1.0mm, F.Cu at (132.2, 87.8)
- added TP37: BUTTON, TestPoint:TestPoint_Pad_D1.0mm, F.Cu at (99.0, 124.5)
- added TP38: NFC_DI, TestPoint:TestPoint_Pad_D1.0mm, F.Cu at (149.3, 65.3)
- added TP39: NFC_DO, TestPoint:TestPoint_Pad_D1.0mm, F.Cu at (151.9, 65.3)
- added TP40: NFC_CLK, TestPoint:TestPoint_Pad_D1.0mm, F.Cu at (154.5, 65.3)
- added TP41: NFC_CS, TestPoint:TestPoint_Pad_D1.0mm, F.Cu at (157.1, 65.3)
- added TP42: NFC_INT, TestPoint:TestPoint_Pad_D1.0mm, F.Cu at (159.7, 65.3)
- added TP43: RFID_DAT, TestPoint:TestPoint_Pad_D1.0mm, F.Cu at (131.2, 69.9)
- added TP44: RFID_WAKE, TestPoint:TestPoint_Pad_D1.0mm, F.Cu at (127.2, 71.6)
- added TP45: 5V, TestPoint:TestPoint_Pad_D1.0mm, F.Cu at (101.0, 121.1)
- C15: footprint Capacitor_SMD:C_0603_1608Metric -> Capacitor_SMD:C_0402_1005Metric
- C4: value NF -> 1pF
- L1: value NF -> 2.7nH
- L2: value NF -> 3.9nH
- TP13: value USB_DM -> USB_DN
- TP7: value SCL_G2 -> SCL_T1
- TP8: value SDA_G2 -> SDA_T1
- moved TP9 114.5 mm to (105.0, 128.0)
- moved TP10 111.7 mm to (107.2, 128.0)
- moved TP12 106.7 mm to (110.8, 71.7)
- moved TP13 105.0 mm to (113.5, 71.7)
- moved TP4 98.1 mm to (118.7, 120.9)
- moved TP3 97.1 mm to (119.8, 119.0)
- moved TP1 94.9 mm to (119.6, 126.4)
- moved TP2 94.4 mm to (119.6, 124.4)
- moved TP6 93.4 mm to (128.2, 134.9)
- moved TP7 92.8 mm to (131.8, 131.7)
- moved R9 92.3 mm to (98.4, 67.5), turned to 90 degrees
- moved TP5 91.5 mm to (130.8, 134.9)
- moved TP8 90.0 mm to (134.0, 130.9)
- moved R8 89.1 mm to (101.3, 67.5), turned to -90 degrees
- moved C4 83.3 mm to (106.8, 136.4), turned to 180 degrees
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Connections:
- C22 pad 1: +3V3_G2 -> /touch/+3V3_G2_IN
- C23 pad 1: +3V3_G2 -> /touch/+3V3_G2_IN
- C24 pad 1: +3V3_G2 -> /touch/+3V3_G2_IN
- C25 pad 1: +3V3_G2 -> /touch/+3V3_G2_IN
- C26 pad 1: VBAT -> /interface/HAPTIC_VBAT_IN
- C27 pad 1: VBAT -> Net-(JP22-B)
- C29 pad 1: +9V -> Net-(D1-A)
- C30 pad 1: +9V -> Net-(D1-A)
- C32 pad 1: VBAT -> Net-(JP32-B)
- C33 pad 1: +3V3 -> /interface/ACC_3V3_IN
- C34 pad 1: +3V3 -> /interface/ACC_3V3_IN
- C35 pad 1: +3V3 -> /interface/ACC_3V3_IN
- C37 pad 1: +5V -> Net-(JP31-A)
- C44 pad 1: +3V3 -> /rf/NFC_3V3_IN
- C51 pad 1: +3V3 -> /rf/NFC_3V3_IN
- C52 pad 1: +3V3 -> /rf/NFC_3V3_IN
- C53 pad 1: +3V3 -> /rf/NFC_3V3_IN
- C54 pad 1: +3V3 -> /rf/NFC_3V3_IN
- C6 pad 1: VBUS_RAW -> /usb/VBUS_RAW
- C7 pad 1: VBUS -> Net-(JP2-A)
- D1 pad 2: +9V -> Net-(D1-A)
- J2 pad 11: VBUS_RAW -> /usb/VBUS_RAW
- J2 pad 2: VBUS_RAW -> /usb/VBUS_RAW
- J5 pad 1: +9V -> unconnected-(J5-NC-Pad1)
- J5 pad 10: OLED_DAT -> /interface/+3V3_G2_IN
- J5 pad 11: GND -> Net-(J5-VCOMH)
- J5 pad 12: unconnected-(J5-NC-Pad12) -> +9V
- J5 pad 2: Net-(J5-VCOMH) -> GND
- J5 pad 3: +3V3_G2 -> /interface/OLED_DAT_IN
- J5 pad 4: GND -> /interface/OLED_CLK_IN
- J5 pad 5: Net-(J5-IREF) -> /interface/OLED_DC_IN
- J5 pad 6: OLED_CS -> /interface/OLED_RST_IN
- J5 pad 7: OLED_RST -> /interface/OLED_CS_IN
- J5 pad 8: OLED_DC -> Net-(J5-IREF)
- J5 pad 9: OLED_CLK -> GND
- L4 pad 1: VBAT -> Net-(JP22-B)
- LED1 pad 1: +5V -> GND
- LED1 pad 3: GND -> +5V
- LED1 pad 4: LED_DAT -> /interface/LED_DAT_IN
- Q1 pad 1: RF_DAT -> /rf/RFID_DAT_IN
- R10 pad 1: +3V3_G2 -> /touch/+3V3_G2_IN
- R10 pad 2: SDA_T1 -> Net-(JP19-B)
- R11 pad 1: +3V3_G2 -> /touch/+3V3_G2_IN
- R11 pad 2: SDA_T2 -> Net-(JP21-B)
- R12 pad 1: +3V3_G2 -> /touch/+3V3_G2_IN
- R12 pad 2: SCL_T1 -> Net-(JP18-B)
- R13 pad 1: +3V3_G2 -> /touch/+3V3_G2_IN
- R13 pad 2: SCL_T2 -> Net-(JP20-B)
- R16 pad 1: +9V -> Net-(D1-A)
- R19 pad 1: LED_EN -> /interface/LED_EN_IN
- R21 pad 1: Net-(D2-A) -> Net-(JP42-B)
- R3 pad 1: TOUCH_INT -> /touch/TOUCH_INT_IN
- R3 pad 2: +3V3_G2 -> /touch/+3V3_G2_IN
- R5 pad 1: VBUS_RAW -> /usb/VBUS_RAW
- R6 pad 1: +3V3 -> /usb/USB_3V3_IN
- R6 pad 2: OVP_FAULT -> Net-(JP1-A)
- TP13 pad 1: USB_DM -> USB_DN
- TP7 pad 1: SCL_G2 -> SCL_T1
- TP8 pad 1: SDA_G2 -> SDA_T1
- U1 pad 25: FUEL_GPOUT -> unconnected-(U1B-PA20-Pad25)
- U1 pad 34: unconnected-(U1B-PA11-Pad34) -> DBG_C
- U1 pad 38: +3V3 -> +3V3_G1
- U1 pad 4: HAPTIC_PWM -> OVP_FAULT
- U1 pad 43: unconnected-(U1B-PA8-Pad43) -> HAPTIC_EN
- U1 pad 44: unconnected-(U1B-PA7-Pad44) -> HAPTIC_PWM
- U1 pad 64: USB_DM -> USB_DN
- U1 pad 7: RF_WAKE -> RFID_WAKE
- U1 pad 8: RF_DAT -> RFID_DAT
- U10 pad 1: SCL -> Net-(JP14-B)
- U10 pad 10: +3V3 -> /interface/ACC_3V3_IN
- U10 pad 12: ACC_INT -> Net-(JP17-A)
- U10 pad 4: SDA -> Net-(JP15-B)
- U10 pad 5: GND -> unconnected-(U10-NC-Pad5)
- U10 pad 9: +3V3 -> /interface/ACC_3V3_IN
- U11 pad 1: +5V -> Net-(JP31-A)
- U11 pad 3: LED_EN -> /interface/LED_EN_IN
- U11 pad 5: VBAT -> Net-(JP32-B)
- U12 pad 4: RF_WAKE -> /rf/RFID_WAKE_IN
- U12 pad 5: +3V3 -> /rf/RFID_3V3_IN
- U13 pad 1: +3V3 -> /rf/NFC_3V3_IN
- U13 pad 10: +3V3 -> /rf/NFC_3V3_IN
- U13 pad 27: NFC_INT -> /rf/NFC_INT_IN
- U13 pad 29: NFC_CS -> /rf/NFC_CS_IN
- U13 pad 30: NFC_CLK -> /rf/NFC_CLK_IN
- U13 pad 31: NFC_DO -> /rf/NFC_DO_IN
- U13 pad 32: NFC_DI -> /rf/NFC_DI_IN
- U13 pad 8: +3V3 -> /rf/NFC_3V3_IN
- U3 pad 1: VBUS -> Net-(JP2-A)
- U3 pad 3: OVP_FAULT -> Net-(JP1-A)
- U3 pad 6: VBUS_RAW -> /usb/VBUS_RAW
- U4 pad 1: /usb/USB_IN_DP -> /usb/USB_IN_DN
- U4 pad 3: /usb/USB_IN_DM -> /usb/USB_IN_DP
- U4 pad 4: USB_DM -> /usb/USB_PROT_DP
- U4 pad 5: VBUS -> /usb/VBUS_RAW
- U4 pad 6: USB_DP -> /usb/USB_PROT_DN
- U5 pad 4: DBG_B -> Net-(JP6-A)
- U5 pad 5: +3V3 -> /usb/USB_3V3_IN
- U5 pad 6: DBG_A -> Net-(JP5-A)
- U6 pad 1: TOUCH_INT -> /touch/TOUCH_INT_IN
- U6 pad 2: SDA_T1 -> Net-(JP19-B)
- U6 pad 3: SCL_T1 -> Net-(JP18-B)
- U6 pad 4: +3V3_G2 -> /touch/+3V3_G2_IN
- U7 pad 1: TOUCH_INT -> /touch/TOUCH_INT_IN
- U7 pad 10: Net-(J4-Pin_7) -> Net-(J4-Pin_2)
- U7 pad 11: Net-(J4-Pin_6) -> Net-(J4-Pin_3)
- U7 pad 12: Net-(J4-Pin_5) -> Net-(J4-Pin_4)
- U7 pad 13: Net-(J4-Pin_4) -> Net-(J4-Pin_5)
- U7 pad 14: Net-(J4-Pin_3) -> Net-(J4-Pin_6)
- U7 pad 15: Net-(J4-Pin_2) -> Net-(J4-Pin_7)
- U7 pad 16: Net-(J4-Pin_1) -> Net-(J4-Pin_8)
- U7 pad 2: SDA_T2 -> Net-(JP21-B)
- U7 pad 3: SCL_T2 -> Net-(JP20-B)
- U7 pad 4: +3V3_G2 -> /touch/+3V3_G2_IN
- U7 pad 9: Net-(J4-Pin_8) -> Net-(J4-Pin_1)
- U8 pad 1: +3V3 -> Net-(JP27-B)
- U8 pad 2: HAPTIC_PWM -> Net-(JP26-B)
- U8 pad 3: +3V3 -> /interface/HAPTIC_VBAT_IN
- U8 pad 7: VBAT -> /interface/HAPTIC_VBAT_IN
- U9 pad 4: OLED_EN -> /interface/OLED_EN_IN
- U9 pad 5: VBAT -> Net-(JP22-B)
Routing:
- net GND: track 0.00 -> 102.7 mm, vias 0 -> 128
- net VBAT: track 0.00 -> 91.4 mm, vias 0 -> 11
- net USB_DP: track 0.00 -> 87.4 mm, vias 0 -> 2
- net USB_DN: track 0.00 -> 85.8 mm, vias 0 -> 2
- net VBUS: track 0.00 -> 77.4 mm, vias 0 -> 2
- net RFID_WAKE: track 0.00 -> 73.2 mm, vias 0 -> 2
- net +3V3_G2: track 0.00 -> 72.7 mm, vias 0 -> 3
- net /interface/OLED_EN_IN: track 0.00 -> 67.1 mm
- net LED_DAT: track 0.00 -> 66.5 mm, vias 0 -> 4
- net RFID_DAT: track 0.00 -> 65.5 mm, vias 0 -> 2
- net LED_EN: track 0.00 -> 55.5 mm, vias 0 -> 2
- net HAPTIC_PWM: track 0.00 -> 52.0 mm, vias 0 -> 2
- net HAPTIC_EN: track 0.00 -> 50.3 mm, vias 0 -> 2
- net /interface/+3V3_G2_IN: track 0.00 -> 45.7 mm
- net +3V3: track 0.00 -> 42.4 mm, vias 0 -> 10
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- added copper zone on In2.Cu, net +3V3
- added copper zone on In2.Cu, net +3V3_G1
- added copper zone on In2.Cu, net /interface/ACC_3V3_IN
- added copper zone on In2.Cu, net /interface/HAPTIC_VBAT_IN
- added copper zone on In2.Cu, net /rf/NFC_3V3_IN
- added copper zone on In2.Cu, net /touch/+3V3_G2_IN
- added copper zone on In2.Cu, net /usb/VBUS_RAW
- added copper zone on F.Cu, net GND
- added copper zone on In1.Cu, net GND
- added copper zone on F.Cu, net VBAT
- added copper zone on In2.Cu, net VBAT
Other:
- board size 58 x 18 mm -> 100 x 80 mm
- copper layers 2 -> 4
- board text added: "(15mm x 15mm)"
- board text added: "(35mm x 20mm)"
- board text added: "(36mm x 17mm)"
- board text added: "(8mm)"
- board text added: "1462360151"
- board text added: "ACC"
- board text added: "ANT"
- board text added: "BAT"
- board text added: "BTM"
- board text added: "Charm BentoBoard"
- board text added: "GY64128-13-C12"
- board text added: "HAPTIC"
- board text added: "LED"
- board text added: "LRA"
- board text added: "NFC"
- board text added: "OLED"
- board text added: "RFID"
- board text added: "Rev1"
- board text added: "TM"
- board text added: "TOP"
- board text added: "TOUCH"
- board text added: "USB"

Commit message: rev1 done hopefully
Parts:
- moved TP23 3.85 mm to (118.3, 109.6)
- moved TP1 3.54 mm to (120.6, 123.0)
- moved TP22 2.20 mm to (118.7, 115.1)
- moved TP2 1.78 mm to (118.5, 123.0)
Connections:
- U1 pad 38: +3V3_G1 -> GND
- U1 pad 4: OVP_FAULT -> unconnected-(U1B-PA29-Pad4)
- U1 pad 50: unconnected-(U1B-PA1-Pad50) -> OVP_FAULT
Routing:
- net NFC_CLK: track 5.82 -> 129.2 mm, vias 2 -> 4
- net NFC_DO: track 6.27 -> 129.2 mm, vias 2 -> 4
- net NFC_DI: track 6.21 -> 129.1 mm, vias 2 -> 4
- net NFC_CS: track 6.53 -> 129.2 mm, vias 2 -> 4
- net NFC_INT: track 4.81 -> 118.0 mm
- net OLED_CLK: track 4.71 -> 105.5 mm, vias 1 -> 2
- net OLED_DAT: track 5.32 -> 105.5 mm, vias 1 -> 2
- net OLED_DC: track 5.22 -> 105.4 mm, vias 1 -> 2
- net OLED_RST: track 4.80 -> 100.9 mm, vias 1 -> 2
- net OLED_CS: track 4.87 -> 94.0 mm, vias 1 -> 2
- net OVP_FAULT: track 1.05 -> 84.4 mm, vias 1 -> 4
- net OLED_EN: track 4.55 -> 87.8 mm, vias 1 -> 2
- net SDA: track 10.4 -> 83.8 mm, vias 1 -> 2
- net DBG_A: track 7.42 -> 79.8 mm, vias 2 -> 4
- net ACC_INT: track 1.41 -> 72.8 mm, vias 1 -> 2
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Other:
- board text added: "Made with <3 by Walter Min"
- board text added: "Rev1 (2026-03-16)"
- board text removed: "Rev1"
