File: rc_keychain.kicad_pcb (KiCad board)
At the start: 4 copper layers, 58 x 18 mm, 144 parts, among them J2 TYPE-C 16PIN 2MD(073), J3 Touch_Surface_Top, J4 Touch_Surface_Bottom, J5 5034801200, Q1 2N7002, SW1 TS35CA, U1 SF32LB525UC6, U10 LIS3DH, U11 AP3602AKTR-G1, U12 SN74AUP1G17, U13 ST25R3916B-AQET, U2 GD25Q256EWIGR, U3 TPS25200DRVT, U4 USBLC6-2P6, U5 USBLC6-2P6, U6 CAP1208-1-A4-TR, U7 CAP1208-1-A4-TR, U8 DRV2603RUNT, U9 TPS61040DBV, Y1 48MHz, Y2 32.768khz, Y3 27.12MHz

Commit message: progress 2
Parts:
- C38, C39, C6, D4, R20, R21, R22, R8, R9, U12, U3: moved to B.Cu
- C7: footprint Capacitor_SMD:C_0603_1608Metric -> Capacitor_SMD:C_0402_1005Metric; moved to B.Cu
- D2: value BAT54WS -> RB521S30T1G; footprint Diode_SMD:D_SOD-323F -> Diode_SMD:D_SOD-523; moved to B.Cu
- D3: value BZT52B3V3 -> BZX584C3V3; footprint Diode_SMD:D_SOD-123 -> Diode_SMD:D_SOD-523; moved to B.Cu
- Q1: value 2N7002 -> 2N7002T; footprint Package_TO_SOT_SMD:SOT-23 -> Package_TO_SOT_SMD:SOT-523; moved to B.Cu
- R23, R5, R6, R7: footprint Resistor_SMD:R_0603_1608Metric -> Resistor_SMD:R_0402_1005Metric; moved to B.Cu
- moved L6 117.2 mm to (44.1, 130.1)
- moved R23 115.3 mm to (48.3, 92.8)
- moved D3 113.9 mm to (50.0, 97.2), turned to 90 degrees
- moved Q1 108.6 mm to (50.5, 92.2), turned to 180 degrees
- moved R22 106.8 mm to (48.3, 95.8), turned to 180 degrees
- moved U12 106.5 mm to (51.9, 97.2), turned to 90 degrees
- moved R20 106.5 mm to (48.3, 94.8), turned to 180 degrees
- moved R21 106.4 mm to (48.3, 97.8)
- moved C38 106.0 mm to (48.3, 93.8), turned to 180 degrees
- moved C39 105.8 mm to (48.3, 96.8)
- moved D2 100.4 mm to (50.0, 94.6), turned to 90 degrees
- moved TP12 100.4 mm to (29.6, 118.2)
- moved TP13 100.4 mm to (29.6, 121.3)
- moved R8 93.9 mm to (40.8, 111.7), turned to -90 degrees
- moved R9 93.9 mm to (40.8, 113.7), turned to -90 degrees
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Connections:
- U5 pad 5: /usb/USB_3V3_IN -> +3V3
Routing:
- net USB_DN: track 0.00 -> 22.6 mm, vias 0 -> 2
- net USB_DP: track 0.00 -> 21.1 mm, vias 0 -> 2
- net GND: track 8.14 -> 23.2 mm, vias 18 -> 28
- net /usb/VBUS_RAW: track 0.00 -> 14.2 mm
- net Net-(C2-Pad2): track 1.26 -> 13.8 mm
- net Net-(J2-CC2): track 0.00 -> 9.90 mm, vias 0 -> 2
- net TOUCH_INT: track 0.00 -> 8.81 mm, vias 1 -> 0
- net FLASH_CS: track 4.84 -> 12.6 mm
- net FLASH_DIO3: track 12.5 -> 5.12 mm
- net /usb/DBG_A_IN: track 0.00 -> 7.20 mm, vias 0 -> 2
- net FLASH_DIO1: track 4.04 -> 11.2 mm
- net FLASH_CLK: track 10.7 -> 3.72 mm
- net FLASH_DIO0: track 8.00 -> 2.30 mm
- net FLASH_DIO2: track 2.66 -> 8.34 mm
- net Net-(J2-CC1): track 0.00 -> 5.38 mm, vias 0 -> 2
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Other:
- board size 58 x 18 mm -> 63 x 18 mm

Commit message: progress 3
Parts:
- C31, C33, C34, C35, R17, R18, SW1, U10: moved to B.Cu
- moved C31 69.4 mm to (54.7, 108.5), turned to -90 degrees
- moved R18 67.6 mm to (53.7, 108.5), turned to -90 degrees
- moved TP37 66.9 mm to (58.9, 102.9)
- moved R17 65.2 mm to (55.7, 108.5), turned to 90 degrees
- moved U6 47.1 mm to (100.3, 107.3), turned to 90 degrees
- moved U7 46.2 mm to (100.3, 118.7), turned to 180 degrees
- moved U10 32.5 mm to (54.0, 118.2), turned to 180 degrees
- moved C33 29.9 mm to (55.3, 115.4), turned to 90 degrees
- moved SW1 28.5 mm to (55.1, 105.5), turned to 180 degrees
- moved C34 28.2 mm to (54.3, 115.4), turned to 90 degrees
- moved C35 26.5 mm to (53.3, 115.4), turned to 90 degrees
- moved L6 19.3 mm to (51.7, 112.3), turned to 90 degrees
- moved C38 17.7 mm to (51.3, 111.2), turned to -90 degrees
- moved C39 17.6 mm to (51.8, 114.1)
- moved R22 17.6 mm to (51.8, 113.1)
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Routing:
- net VBUS: track 72.6 -> 3.81 mm
- net +3V3_G2: track 67.2 -> 2.15 mm, vias 2 -> 1
- net Net-(J4-Pin_8): track 0.00 -> 39.6 mm
- net Net-(J3-Pin_1): track 0.00 -> 38.5 mm
- net Net-(J4-Pin_7): track 0.00 -> 34.4 mm
- net Net-(J3-Pin_2): track 0.00 -> 34.4 mm
- net Net-(J4-Pin_6): track 0.00 -> 29.2 mm
- net Net-(J3-Pin_3): track 0.00 -> 29.2 mm
- net Net-(J4-Pin_5): track 0.00 -> 24.0 mm
- net Net-(J3-Pin_4): track 0.00 -> 24.0 mm
- net Net-(J4-Pin_4): track 0.00 -> 19.4 mm
- net Net-(J3-Pin_5): track 0.00 -> 19.4 mm
- net VBAT: track 24.5 -> 7.63 mm
- net Net-(J4-Pin_3): track 0.00 -> 15.1 mm
- net Net-(J3-Pin_6): track 0.00 -> 15.1 mm
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- added copper zone on In1.Cu, net +3V3
- removed copper zone on In2.Cu, net (none)
- removed copper zone on In2.Cu, net +3V3
- removed copper zone on In2.Cu, net +3V3_G1
- removed copper zone on In2.Cu, net /usb/VBUS_RAW
- removed copper zone on In1.Cu, net GND
- removed copper zone on In2.Cu, net VBAT

Commit message: progress 4
Parts:
- BT1: moved to B.Cu
- moved BT1 38.0 mm to (57.0, 119.3), turned to 90 degrees
- moved U12 16.0 mm to (55.4, 113.3)
- moved R21 0.93 mm to (53.4, 113.4), turned to -90 degrees
- moved Y2 0.23 mm to (57.0, 115.8)
- moved R23 0.15 mm to (51.7, 109.5)
- moved Q1 0.14 mm to (51.5, 107.8)
- moved D2 0.05 mm to (53.6, 110.8)
- moved D3 0.05 mm to (55.1, 110.8)
- turned C5 to 90 degrees
Routing:
- net VBUS: track 3.81 -> 18.6 mm, vias 1 -> 2
- net RFID_DAT: track 1.96 -> 14.5 mm, vias 1 -> 2
- net VBAT: track 7.63 -> 19.4 mm
- net SCL: track 1.13 -> 12.2 mm, vias 1 -> 2
- net SDA: track 1.30 -> 11.5 mm, vias 1 -> 2
- net GND: track 24.5 -> 32.6 mm, vias 28 -> 33
- net RFID_WAKE: track 2.13 -> 7.69 mm, vias 1 -> 2
- net +3V3: track 3.97 -> 9.06 mm, vias 3 -> 6
- net +3V3_G1: track 3.40 -> 8.31 mm, vias 1 -> 2
- net Net-(D3-K): track 0.00 -> 3.43 mm
- net Net-(Q1-D): track 0.00 -> 1.39 mm
- net Net-(D2-K): track 3.23 -> 4.01 mm
- net USB_DN: track 22.6 -> 23.2 mm
- net ACC_INT: track 0.82 -> 1.46 mm, vias 1 -> 2
- net NFC_DI: track 2.09 -> 2.68 mm
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