File: rc_keychain.kicad_pcb (KiCad board)
At the start: 4 copper layers, 63 x 18 mm, 144 parts, among them J2 TYPE-C 16PIN 2MD(073), J3 Touch_Surface_Top, J4 Touch_Surface_Bottom, J5 5034801200, Q1 2N7002T, SW1 TS35CA, U1 SF32LB525UC6, U10 LIS3DH, U11 AP3602AKTR-G1, U12 SN74AUP1G17, U13 ST25R3916B-AQET, U2 GD25Q256EWIGR, U3 TPS25200DRVT, U4 USBLC6-2P6, U5 USBLC6-2P6, U6 CAP1208-1-A4-TR, U7 CAP1208-1-A4-TR, U8 DRV2603RUNT, U9 TPS61040DBV, Y1 48MHz, Y2 32.768khz, Y3 27.12MHz

Commit message: progress 5
Parts:
- C22, C23, C24, C25, C26, C27, C28, C29, C30, C32, C36, C37, C40, C41, C42, C43, C44, C45, C46, C47, C48, C49, C50, C51, C52, C53, C54, C55, C56, C57, C58, C59, C60, C61, D1, L4, L5, L7, L8, LED1, R10, R11, R12, R13, R14, R15, R16, R19, R2, R24, R4, U11, U13, U8, U9, Y3: moved to B.Cu
- moved R4 40.6 mm to (49.1, 116.4)
- moved R2 37.9 mm to (49.1, 117.5)
- moved C30 32.7 mm to (107.6, 133.3), turned to 180 degrees
- moved TP15 29.2 mm to (56.7, 98.4)
- moved TP14 29.2 mm to (56.7, 95.3)
- moved L4 24.5 mm to (112.0, 125.5), turned to 180 degrees
- moved U11 24.3 mm to (112.0, 129.6), turned to 180 degrees
- moved C42 23.5 mm to (106.3, 90.3), turned to 180 degrees
- moved C43 23.5 mm to (106.3, 92.1), turned to 180 degrees
- moved C44 23.5 mm to (106.3, 93.8), turned to 180 degrees
- moved C45 23.5 mm to (106.3, 95.6), turned to 180 degrees
- moved C46 23.5 mm to (106.3, 97.3), turned to 180 degrees
- moved C47 23.5 mm to (106.3, 99.1), turned to 180 degrees
- moved U8 23.4 mm to (112.5, 133.8), turned to 180 degrees
- moved C48 18.6 mm to (103.8, 90.3), turned to 180 degrees
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Routing:
- net ACC_INT: track 1.46 -> 14.5 mm
- net SCL: track 12.2 -> 21.4 mm
- net SDA: track 11.5 -> 16.9 mm
- net +3V3: track 9.06 -> 11.6 mm, vias 6 -> 8
- net GND: track 32.6 -> 30.2 mm, vias 33 -> 38
- net SDA_T2: track 0.97 -> 0.00 mm, vias 1 -> 0
- net SDA_T1: track 0.91 -> 0.00 mm, vias 1 -> 0
- net SCL_T2: track 0.89 -> 0.00 mm, vias 1 -> 0
- net BUTTON: track 4.23 -> 5.03 mm, vias 1 -> 2
- net VBAT: track 19.4 -> 19.6 mm, vias 2 -> 3

Commit message: progress before minor redesign
Parts:
- removed C32, C37: 10uF, Capacitor_SMD:C_0402_1005Metric
- removed C36: 1uF, Capacitor_SMD:C_0402_1005Metric
- removed LED1: XL-4020RGBC-WS2812B, XL-4020RGBC-2812B:LED-SMD_4P-L4.0-W1.7_XL-4020RGBC-WS2812B
- removed R19: 100k, Resistor_SMD:R_0402_1005Metric
- removed TP45: 5V, TestPoint:TestPoint_Pad_D1.0mm
- removed U11: AP3602AKTR-G1, AP3602AKTR-G1:SOT-23-6_L2.9-W1.6-P0.95-LS2.8-BR
- added D5: KT-0805G, Diode_SMD:D_0805_2012Metric, F.Cu at (99.8, 135.5)
- added R1: 100, Resistor_SMD:R_0402_1005Metric, F.Cu at (99.0, 138.0)
- moved TP37 5.41 mm to (61.2, 98.0)
- moved L8 2.88 mm to (88.5, 81.5)
- moved J5 0.33 mm to (99.7, 113.0)
Routing:
- net +3V3: track 11.6 -> 10.4 mm, vias 8 -> 6
- net BUTTON: track 5.03 -> 4.42 mm, vias 2 -> 1

Commit message: progress before stepping
Parts:
- SW1: value TS35CA -> HX 3X4X2-2P-1.6N; footprint TS35CA:KEY-SMD_TS35CA -> HX3x4x2-2P-1:KEY-SMD_L4.0-W3.0-LS4.9-1
- moved R21 8.36 mm to (51.8, 105.2), turned to 0 degrees
- moved D3 8.18 mm to (54.4, 102.7), turned to 180 degrees
- moved U12 7.88 mm to (54.2, 105.5)
- moved SW1 7.68 mm to (53.7, 113.0)
- moved C39 5.91 mm to (55.1, 109.2), turned to 90 degrees
- moved R22 4.52 mm to (54.1, 109.2), turned to -90 degrees
- moved C31 3.73 mm to (51.8, 110.8), turned to 180 degrees
- moved L6 3.64 mm to (53.6, 109.2), turned to 180 degrees
- moved D2 3.49 mm to (54.1, 107.4), turned to 180 degrees
- moved R20 2.53 mm to (52.6, 108.7), turned to 0 degrees
- moved R18 2.31 mm to (53.7, 110.8), turned to 0 degrees
- moved R17 2.30 mm to (55.6, 110.8), turned to 0 degrees
- moved C38 1.98 mm to (52.6, 109.7), turned to 0 degrees
- moved Q1 0.83 mm to (51.7, 106.9)
- moved R23 0.67 mm to (51.1, 109.2), turned to 90 degrees
Routing:
- net BUTTON: track 4.42 -> 22.6 mm, vias 1 -> 2
- net RFID_DAT: track 14.5 -> 1.96 mm, vias 2 -> 1
- net RFID_WAKE: track 7.69 -> 2.13 mm, vias 2 -> 1
- net Net-(D3-K): track 3.43 -> 0.00 mm
- net Net-(D2-K): track 4.01 -> 7.44 mm
- net GND: track 30.2 -> 29.5 mm, vias 38 -> 37
- net Net-(D2-A): track 4.60 -> 5.29 mm
- net VBUS: track 18.6 -> 18.0 mm
- net +3V3: track 10.4 -> 9.88 mm, vias 6 -> 5

Commit message: progress before restarting bigtime
Parts:
- moved R1 51.0 mm to (53.7, 114.6), turned to 180 degrees
- moved D5 50.9 mm to (54.1, 113.0)
- moved D3 3.21 mm to (54.2, 105.9), turned to 0 degrees
- moved U12 2.82 mm to (56.9, 106.3)
- moved L6 0.76 mm to (53.9, 109.9)
- moved R21 0.10 mm to (51.7, 105.2)
- turned J5 to -90 degrees
Connections:
- U1 pad 4: unconnected-(U1B-PA29-Pad4) -> TOUCH_INT
- U1 pad 5: LED_EN -> unconnected-(U1B-PA28-Pad5)
- U1 pad 6: TOUCH_INT -> unconnected-(U1B-PA27-Pad6)
Routing:
- net RFID_DAT: track 1.96 -> 15.6 mm, vias 1 -> 2
- net RFID_WAKE: track 2.13 -> 11.9 mm, vias 1 -> 2
- net Net-(D3-K): track 0.00 -> 4.40 mm
- net LED_DAT: track 1.74 -> 5.93 mm
- net SCL_T2: track 0.00 -> 3.73 mm, vias 0 -> 1
- net SDA_T1: track 0.00 -> 3.69 mm, vias 0 -> 1
- net GND: track 29.5 -> 32.1 mm, vias 37 -> 40
- net SDA_T2: track 0.00 -> 2.33 mm, vias 0 -> 1
- net TOUCH_INT: track 0.00 -> 2.31 mm, vias 0 -> 1
- net Net-(D5-K): track 0.00 -> 1.61 mm
- net Net-(D2-A): track 5.29 -> 6.37 mm
- net VBUS: track 18.0 -> 18.7 mm
- net BUTTON: track 22.6 -> 23.1 mm
- net +3V3: track 9.88 -> 10.4 mm, vias 5 -> 6
