File: mcu.kicad_sch (KiCad schematic)
At the start: 34 parts, among them J1 U.FL-R-SMT-1(10), U1 SF32LB525UC6, U2 MKDV1GCL-ABA, Y1 48MHz, Y2 32.768khz

Commit message: huge progress on bentoboard, schematic fixes
Parts:
- removed R3: 100k, Resistor_SMD:R_0402_1005Metric, symbol Device:R_Small
Connections:
- net DBG_B: no longer TP25.1
- net DBG_C: now also TP25.1
Changed lines of the file:
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@@
 	)
 	(junction
-		(at 152.4 78.74)
-		(diameter 0)
-		(color 0 0 0 0)
-	)
-	(junction
 		(at 148.59 50.8)
 		(diameter 0)
@@
 	(wire
 		(pts
-			(xy 152.4 76.2) (xy 152.4 78.74)
-		)
-		(stroke
-			(width 0)
-			(type default)
-		)
-	)
-	(wire
-		(pts
 			(xy 166.37 106.68) (xy 168.91 106.68)
 		)
@@
 	(wire
 		(pts
-			(xy 158.75 76.2) (xy 163.83 76.2)
-		)
-		(stroke
-			(width 0)
-			(type default)
-		)
-	)
-	(wire
-		(pts
 			(xy 148.59 50.8) (xy 148.59 52.07)
 		)
@@
 	(wire
 		(pts
-			(xy 152.4 78.74) (xy 154.94 78.74)
-		)
-		(stroke
-			(width 0)
-			(type default)
-		)
-	)
-	(wire
-		(pts
 			(xy 100.33 139.7) (xy 106.68 139.7)
 		)
@@
 	(wire
 		(pts
-			(xy 153.67 76.2) (xy 152.4 76.2)
-		)
-		(stroke
-			(width 0)
-			(type default)
-		)
-	)
-	(wire
-		(pts
 			(xy 256.54 111.76) (xy 252.73 111.76)
 		)
@@
 	(wire
 		(pts
-			(xy 137.16 78.74) (xy 152.4 78.74)
-		)
-		(stroke
-			(width 0)
-			(type default)
-		)
-	)
-	(wire
-		(pts
 			(xy 101.6 124.46) (xy 106.68 124.46)
 		)
@@
 		)
 	)
+	(global_label "TOUCH_INT"
+		(shape input)
+		(at 137.16 78.74 0)
+		(fields_autoplaced yes)
+		(effects
+			(font
+				(size 1.27 1.27)
+			)
+			(justify left)
+		)
+		(property "Intersheetrefs" "${INTERSHEET_REFS}"
+			(at 150.2448 78.74 0)
+			(effects
+				(font
+					(size 1.27 1.27)
+				)
+				(justify left)
+				(hide yes)
+			)
+		)
+	)
 	(global_label "OLED_DAT"
 		(shape input)
@@
 		)
 	)
-	(global_label "DBG_B"
+	(global_label "DBG_C"
 		(shape input)
 		(at 46.99 124.46 180)
@@
 		)
 	)
-	(global_label "TOUCH_INT"
-		(shape input)
-		(at 154.94 78.74 0)
-		(fields_autoplaced yes)
-		(effects
-			(font
-				(size 1.27 1.27)
-			)
-			(justify left)
-		)
-		(property "Intersheetrefs" "${INTERSHEET_REFS}"
-			(at 168.0248 78.74 0)
-			(effects
-				(font
-					(size 1.27 1.27)
-				)
-				(justify left)
-				(hide yes)
-			)
-		)
-	)
 	(global_label "SDA"
 		(shape input)
@@
 	)
 	(symbol
-		(lib_id "custom_syms:+3V3_G2")
-		(at 163.83 76.2 0)
-		(unit 1)
-		(exclude_from_sim no)
-		(in_bom yes)
-		(on_board yes)
-		(dnp no)
-		(property "Reference" "#PWR09"
-			(at 163.83 80.01 0)
-			(effects
-				(font
-					(size 1.27 1.27)
-				)
-				(hide yes)
-			)
-		)
-		(property "Value" "+3V3_G2"
-			(at 163.83 72.644 0)
-			(effects
-				(font
-					(size 1.27 1.27)
-				)
-			)
-		)
-		(property "Footprint" ""
-			(at 163.83 76.2 0)
-			(effects
-				(font
-					(size 1.27 1.27)
-				)
-				(hide yes)
-			)
-		)
-		(property "Datasheet" ""
-			(at 163.83 76.2 0)
-			(effects
-				(font
-					(size 1.27 1.27)
-				)
-				(hide yes)
-			)
-		)
-		(property "Description" "Power symbol creates a global label with name \"+3V3_G2\""
-			(at 163.83 76.2 0)
-			(effects
-				(font
-					(size 1.27 1.27)
-				)
-				(hide yes)
-			)
-		)
-		(pin "1"
-		)
-		(instances
-			(project ""
-				(path "/c6cb5a1d-9f97-4766-8582-a9e93ed049e4/c4c0fb03-7c4b-4d55-99ac-6edbef8e602c"
-					(reference "#PWR09")
-					(unit 1)
-				)
-			)
-		)
-	)
-	(symbol
 		(lib_id "Connector:TestPoint")
 		(at 46.99 100.33 270)
@@
 					(size 1.27 1.27)
 				)
+				(hide yes)
 			)
 		)
@@
 					(unit 1)
 				)
-			)
-		)
-	)
-	(symbol
-		(lib_id "Device:R_Small")
-		(at 156.21 76.2 90)
-		(unit 1)
-		(exclude_from_sim no)
-		(in_bom yes)
-		(on_board yes)
-		(dnp no)
-		(property "Reference" "R3"
-			(at 156.21 72.644 90)
-			(effects
-				(font
-					(size 1.016 1.016)
-				)
-			)
-		)
-		(property "Value" "100k"
-			(at 156.21 74.422 90)
-			(effects
-				(font
-					(size 1.27 1.27)
-				)
-			)
-		)
-		(property "Footprint" "Resistor_SMD:R_0402_1005Metric"
-			(at 156.21 76.2 0)
-			(effects
-				(font
-					(size 1.27 1.27)
-				)
-				(hide yes)
-			)
-		)
-		(property "Datasheet" "~"
-			(at 156.21 76.2 0)
-			(effects
-				(font
-					(size 1.27 1.27)
-				)
-				(hide yes)
-			)
-		)
-		(property "Description" "Resistor, small symbol"
-			(at 156.21 76.2 0)
-			(effects
-				(font
-					(size 1.27 1.27)
-				)
-				(hide yes)
-			)
-		)
-		(property "LCSC Part" "C25741"
-			(at 156.21 76.2 90)
-			(effects
-				(font
-					(size 1.27 1.27)
-				)
-				(hide yes)
-			)
-		)
-		(property "CREATOR" ""
-			(at 156.21 76.2 90)
-			(effects
-				(font
-					(size 1.27 1.27)
-				)
-				(hide yes)
-			)
-		)
-		(property "MAXIMUM_PACKAGE_HEIGHT" ""
-			(at 156.21 76.2 90)
-			(effects
-				(font
-					(size 1.27 1.27)
-				)
-				(hide yes)
-			)
-		)
-		(property "PARTREV" ""
-			(at 156.21 76.2 90)
-			(effects
-				(font
-					(size 1.27 1.27)
-				)
-				(hide yes)
-			)
-		)
-		(property "VERIFIER" ""
-			(at 156.21 76.2 90)
-			(effects
-				(font
-					(size 1.27 1.27)
-				)
-				(hide yes)
-			)
-		)
-		(pin "2"
-		)
-		(pin "1"
-		)
-		(instances
-			(project ""
-				(path "/c6cb5a1d-9f97-4766-8582-a9e93ed049e4/c4c0fb03-7c4b-4d55-99ac-6edbef8e602c"
-					(reference "R3")
-					(unit 1)
-				)

Commit message: rev1 done hopefully
Connections:
- net +3V3_G1: no longer U1.38 (AVDD33_AUD)
- net GND: now also U1.38 (AVDD33_AUD)
- net OVP_FAULT: now also U1.50 (PA1); no longer U1.4 (PA29)
Changed lines of the file:
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@@
 	)
 	(no_connect
-		(at 137.16 129.54)
+		(at 137.16 83.82)
 	)
 	(no_connect
-		(at 106.68 73.66)
+		(at 137.16 129.54)
 	)
 	(wire
@@
 	(global_label "OVP_FAULT"
 		(shape input)
-		(at 137.16 83.82 0)
+		(at 106.68 73.66 180)
 		(fields_autoplaced yes)
 		(effects
@@
 				(size 1.27 1.27)
 			)
-			(justify left)
+			(justify right)
 		)
 		(property "Intersheetrefs" "${INTERSHEET_REFS}"
-			(at 150.3053 83.82 0)
+			(at 93.5347 73.66 0)
 			(effects
 				(font
 					(size 1.27 1.27)
 				)
-				(justify left)
+				(justify right)
 				(hide yes)
 			)
@@
 	)
 	(symbol
+		(lib_id "power:GND")
+		(at 137.16 139.7 90)
+		(unit 1)
+		(exclude_from_sim no)
+		(in_bom yes)
+		(on_board yes)
+		(dnp no)
+		(property "Reference" "#PWR04"
+			(at 143.51 139.7 0)
+			(effects
+				(font
+					(size 1.27 1.27)
+				)
+				(hide yes)
+			)
+		)
+		(property "Value" "GND"
+			(at 140.208 139.7 90)
+			(effects
+				(font
+					(size 1.27 1.27)
+				)
+				(justify right)
+			)
+		)
+		(property "Footprint" ""
+			(at 137.16 139.7 0)
+			(effects
+				(font
+					(size 1.27 1.27)
+				)
+				(hide yes)
+			)
+		)
+		(property "Datasheet" ""
+			(at 137.16 139.7 0)
+			(effects
+				(font
+					(size 1.27 1.27)
+				)
+				(hide yes)
+			)
+		)
+		(property "Description" "Power symbol creates a global label with name \"GND\" , ground"
+			(at 137.16 139.7 0)
+			(effects
+				(font
+					(size 1.27 1.27)
+				)
+				(hide yes)
+			)
+		)
+		(pin "1"
+		)
+		(instances
+			(project ""
+				(path "/c6cb5a1d-9f97-4766-8582-a9e93ed049e4/c4c0fb03-7c4b-4d55-99ac-6edbef8e602c"
+					(reference "#PWR04")
+					(unit 1)
+				)
+			)
+		)
+	)
+	(symbol
 		(lib_id "PCM_MCU_SiFli:SF32LB52xUx")
 		(at 121.92 104.14 0)
@@
 					(unit 1)
 				)
-			)
-		)
-	)
-	(symbol
-		(lib_id "custom_syms:+3V3_G1")
-		(at 137.16 139.7 270)
-		(unit 1)
-		(exclude_from_sim no)
-		(in_bom yes)
-		(on_board yes)
-		(dnp no)
-		(property "Reference" "#PWR04"
-			(at 133.35 139.7 0)
-			(effects
-				(font
-					(size 1.27 1.27)
-				)
-				(hide yes)
-			)
-		)
-		(property "Value" "+3V3_G1"
-			(at 140.208 139.7 90)
-			(effects
-				(font
-					(size 1.27 1.27)
-				)
-				(justify left)
-			)
-		)
-		(property "Footprint" ""
-			(at 137.16 139.7 0)
-			(effects
-				(font
-					(size 1.27 1.27)
-				)
-				(hide yes)
-			)
-		)
-		(property "Datasheet" ""
-			(at 137.16 139.7 0)
-			(effects
-				(font
-					(size 1.27 1.27)
-				)
-				(hide yes)
-			)
-		)
-		(property "Description" "Power symbol creates a global label with name \"+3V3_G1\""
-			(at 137.16 139.7 0)
-			(effects
-				(font
-					(size 1.27 1.27)
-				)
-				(hide yes)
-			)
-		)
-		(pin "1"
-		)
-		(instances
-			(project ""
-				(path "/c6cb5a1d-9f97-4766-8582-a9e93ed049e4/c4c0fb03-7c4b-4d55-99ac-6edbef8e602c"
-					(reference "#PWR04")
-					(unit 1)
-				)

Commit message: fixups before manufacturing pt1
Parts:
- U2: value MKDV1GCL-ABA -> MKDV1GCL-ABF; LCSC Part C6152616 -> C51966230
Changed lines of the file:
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@@
 			)
 		)
-		(property "Value" "MKDV1GCL-ABA"
+		(property "Value" "MKDV1GCL-ABF"
 			(at 233.68 115.57 0)
 			(effects
@@
 			)
 		)
-		(property "LCSC Part" "C6152616"
+		(property "LCSC Part" "C51966230"
 			(at 233.68 138.43 0)
 			(effects

Commit message: fixups before manufacturing pt2
Parts:
- removed R1: 7.5k, Resistor_SMD:R_0603_1608Metric, symbol Device:R_Small
- removed U2: MKDV1GCL-ABF, MKDV1GCL-ABA:LGA-8_L6.0-W8.0-P1.27-TL, symbol MKDV1GCL-ABA:MKDV1GCL-ABA
- added U2: GD25Q256EWIGR, GD25Q256EWIGR:WSON-8_L6.0-W5.0-P1.27-TL-EP, symbol GD25Q256EWIGR:GD25Q256EWIGR
- TP18: value SD_CLK -> FLASH_CLK
- TP19: value SD_CLK -> FLASH_CS
- TP20: value SD_DAT0 -> FLASH_DIO0
- TP21: value SD_DAT1 -> FLASH_DIO1
- TP22: value SD_DAT2 -> FLASH_DIO2
- TP23: value SD_DAT3 -> FLASH_DIO3
Connections:
- net +3V3_G1: now also U2.8 (VCC)
- net GND: now also U2.4 (VSS), U2.9 (EP)
- net SD_CLK renamed FLASH_CLK
- net FLASH_CLK: now also U1.29 (PA16), U2.6 (SCLK); no longer U1.31 (PA14)
- net SD_CMD renamed FLASH_CS
- net FLASH_CS: now also U1.33 (PA12), U2.1 (~{CS}); no longer U1.30 (PA15)
- net SD_DAT0 renamed FLASH_DIO0
- net FLASH_DIO0: now also U1.30 (PA15), U2.5 (SI(IO0)); no longer U1.29 (PA16)
- net SD_DAT1 renamed FLASH_DIO1
- net FLASH_DIO1: now also U1.32 (PA13), U2.2 (SO(IO1)); no longer U1.28 (PA17)
- net SD_DAT2 renamed FLASH_DIO2
- net FLASH_DIO2: now also U1.31 (PA14), U2.3 (WP#(IO2)); no longer U1.33 (PA12)
- net SD_DAT3 renamed FLASH_DIO3
- net FLASH_DIO3: now also U1.28 (PA17), U2.7 (~{HOLD}/RESET#(IO3)); no longer U1.32 (PA13)
Other:
- note removed: "Pull up to configure boot from SD Card"
- moved on the sheet: C5, TP18, TP19, TP20, TP21, TP22, TP23

Commit message: layout progress
Parts:
- removed J1: U.FL-R-SMT-1(10), U.FL-R-SMT-1_10_:HRS_U.FL-R-SMT-1_10_, symbol U.FL-R-SMT-1_10_:U.FL-R-SMT-1_10_
- removed TP18: FLASH_CLK, TestPoint:TestPoint_Pad_D1.0mm, symbol Connector:TestPoint
- removed TP19: FLASH_CS, TestPoint:TestPoint_Pad_D1.0mm, symbol Connector:TestPoint
- removed TP20: FLASH_DIO0, TestPoint:TestPoint_Pad_D1.0mm, symbol Connector:TestPoint
- removed TP21: FLASH_DIO1, TestPoint:TestPoint_Pad_D1.0mm, symbol Connector:TestPoint
- removed TP22: FLASH_DIO2, TestPoint:TestPoint_Pad_D1.0mm, symbol Connector:TestPoint
- removed TP23: FLASH_DIO3, TestPoint:TestPoint_Pad_D1.0mm, symbol Connector:TestPoint

Commit message: progress
Parts:
- removed C1, C3: NF, Capacitor_SMD:C_0402_1005Metric, symbol Device:C_Small
- Y1: footprint Crystal:Crystal_SMD_2520-4Pin_2.5x2.0mm -> Crystal:Crystal_SMD_2016-4Pin_2.0x1.6mm; LCSC Part C2932991 -> C49363531
Other:
- note added: "Remove C2 for VNA"
- note removed: "Remove C2 & C3 for VNA"
- moved on the sheet: C2

Commit message: progress before restarting bigtime
Connections:
- net TOUCH_INT: now also U1.4 (PA29); no longer U1.6 (PA27)
- net LED_EN: no longer names the net of U1.5 (PA28)
- no-connect marks 7 -> 8
Changed lines of the file:
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@@
+	)
+	(no_connect
+		(at 137.16 78.74)
+	)
+	(no_connect
+		(at 137.16 81.28)
 	)
 	(no_connect
@@
 	)
 	(no_connect
-		(at 137.16 83.82)
-	)
-	(no_connect
 		(at 137.16 129.54)
 	)
@@
 	(global_label "TOUCH_INT"
 		(shape input)
-		(at 137.16 78.74 0)
+		(at 137.16 83.82 0)
 		(fields_autoplaced yes)
 		(effects
@@
 		)
 		(property "Intersheetrefs" "${INTERSHEET_REFS}"
-			(at 150.2448 78.74 0)
+			(at 150.2448 83.82 0)
 			(effects
 				(font
@@
 			(effects
 				(font
-					(size 1.27 1.27)
-				)
-				(justify left)
-				(hide yes)
-			)
-		)
-	)
-	(global_label "LED_EN"
-		(shape input)
-		(at 137.16 81.28 0)
-		(fields_autoplaced yes)
-		(effects
-			(font
-				(size 1.27 1.27)
-			)
-			(justify left)
-		)
-		(property "Intersheetrefs" "${INTERSHEET_REFS}"
-			(at 147.0394 81.28 0)
-			(effects
-				(font

Commit message: huge progress
Connections:
- net OLED_EN: no longer names the net of U1.49 (PA2)
- no-connect marks 8 -> 9
Changed lines of the file:
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@@
+	)
+	(no_connect
+		(at 106.68 76.2)
 	)
 	(no_connect
@@
 			(effects
 				(font
-					(size 1.27 1.27)
-				)
-				(justify right)
-				(hide yes)
-			)
-		)
-	)
-	(global_label "OLED_EN"
-		(shape input)
-		(at 106.68 76.2 180)
-		(fields_autoplaced yes)
-		(effects
-			(font
-				(size 1.27 1.27)
-			)
-			(justify right)
-		)
-		(property "Intersheetrefs" "${INTERSHEET_REFS}"
-			(at 95.4701 76.2 0)
-			(effects
-				(font
