File: interface.kicad_sch (KiCad schematic)
At the start: 26 parts, among them J5 5034801200, SW1 TS35CA, U10 LIS3DH, U8 DRV2603RUNT, U9 TPS61040DBV

Commit message: progress before stepping
Parts:
- removed SW1: TS35CA, TS35CA:KEY-SMD_TS35CA, symbol TS35CA:TS35CA
- added SW1: HX 3X4X2-2P-1.6N, HX3x4x2-2P-1:KEY-SMD_L4.0-W3.0-LS4.9-1, symbol HX3x4x2-2P-1:HX3X4X2-2P-1.6NTACTILESWITCH
Connections:
- net BUTTON: now also SW1.2
- net at R17.2: now also SW1.1
- no-connect marks 7 -> 5
Other:
- moved on the sheet: R17
Changed lines of the file:
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@@
 	)
 	(no_connect
-		(at 184.15 82.55)
-	)
-	(no_connect
-		(at 173.99 82.55)
-	)
-	(no_connect
 		(at 59.69 48.26)
 	)
@@
 	(wire
 		(pts
-			(xy 166.37 80.01) (xy 173.99 80.01)
+			(xy 165.1 80.01) (xy 173.99 80.01)
 		)
 		(stroke
@@
 	(wire
 		(pts
-			(xy 166.37 77.47) (xy 166.37 80.01)
+			(xy 165.1 74.93) (xy 165.1 80.01)
 		)
 		(stroke
@@
 	(symbol
 		(lib_id "power:+3V3")
-		(at 166.37 72.39 0)
+		(at 165.1 69.85 0)
 		(unit 1)
 		(exclude_from_sim no)
@@
 		(fields_autoplaced yes)
 		(property "Reference" "#PWR082"
-			(at 166.37 76.2 0)
+			(at 165.1 73.66 0)
 			(effects
 				(font
@@
 		)
 		(property "Value" "+3V3"
-			(at 166.37 67.31 0)
+			(at 165.1 64.77 0)
 			(effects
 				(font
@@
 		)
 		(property "Footprint" ""
-			(at 166.37 72.39 0)
+			(at 165.1 69.85 0)
 			(effects
 				(font
@@
 		)
 		(property "Datasheet" ""
-			(at 166.37 72.39 0)
+			(at 165.1 69.85 0)
 			(effects
 				(font
@@
 		)
 		(property "Description" "Power symbol creates a global label with name \"+3V3\""
-			(at 166.37 72.39 0)
+			(at 165.1 69.85 0)
 			(effects
 				(font
@@
 	)
 	(symbol
-		(lib_id "TS35CA:TS35CA")
-		(at 179.07 80.01 0)
-		(unit 1)
-		(exclude_from_sim no)
-		(in_bom yes)
-		(on_board yes)
-		(dnp no)
-		(fields_autoplaced yes)
-		(property "Reference" "SW1"
-			(at 179.58 73.66 0)
-			(effects
-				(font
-					(size 1.27 1.27)
-				)
-			)
-		)
-		(property "Value" "TS35CA"
-			(at 179.58 76.2 0)
-			(effects
-				(font
-					(size 1.27 1.27)
-				)
-			)
-		)
-		(property "Footprint" "TS35CA:KEY-SMD_TS35CA"
-			(at 179.07 90.17 0)
-			(effects
-				(font
-					(size 1.27 1.27)
-				)
-				(hide yes)
-			)
-		)
-		(property "Datasheet" ""
-			(at 179.07 80.01 0)
-			(effects
-				(font
-					(size 1.27 1.27)
-				)
-				(hide yes)
-			)
-		)
-		(property "Description" ""
-			(at 179.07 80.01 0)
-			(effects
-				(font
-					(size 1.27 1.27)
-				)
-				(hide yes)
-			)
-		)
-		(property "LCSC Part" "C412366"
-			(at 179.07 92.71 0)
-			(effects
-				(font
-					(size 1.27 1.27)
-				)
-				(hide yes)
-			)
-		)
-		(property "CREATOR" ""
-			(at 179.07 80.01 0)
-			(effects
-				(font
-					(size 1.27 1.27)
-				)
-				(hide yes)
-			)
-		)
-		(property "MAXIMUM_PACKAGE_HEIGHT" ""
-			(at 179.07 80.01 0)
-			(effects
-				(font
-					(size 1.27 1.27)
-				)
-				(hide yes)
-			)
-		)
-		(property "PARTREV" ""
-			(at 179.07 80.01 0)
-			(effects
-				(font
-					(size 1.27 1.27)
-				)
-				(hide yes)
-			)
-		)
-		(property "VERIFIER" ""
-			(at 179.07 80.01 0)
-			(effects
-				(font
-					(size 1.27 1.27)
-				)
-				(hide yes)
-			)
-		)
-		(property "AVAILABILITY" ""
-			(at 179.07 80.01 0)
-			(effects
-				(font
-					(size 1.27 1.27)
-				)
-				(hide yes)
-			)
-		)
-		(property "DESCRIPTION" ""
-			(at 179.07 80.01 0)
-			(effects
-				(font
-					(size 1.27 1.27)
-				)
-				(hide yes)
-			)
-		)
-		(property "MANUFACTURER" ""
-			(at 179.07 80.01 0)
-			(effects
-				(font
-					(size 1.27 1.27)
-				)
-				(hide yes)
-			)
-		)
-		(property "PACKAGE" ""
-			(at 179.07 80.01 0)
-			(effects
-				(font
-					(size 1.27 1.27)
-				)
-				(hide yes)
-			)
-		)
-		(property "PRICE" ""
-			(at 179.07 80.01 0)
-			(effects
-				(font
-					(size 1.27 1.27)
-				)
-				(hide yes)
-			)
-		)
-		(property "STANDARD" ""
-			(at 179.07 80.01 0)
-			(effects
-				(font
-					(size 1.27 1.27)
-				)
-				(hide yes)
-			)
-		)
-		(pin "1"
-		)
-		(pin "2"
-		)
-		(pin "4"
-		)
-		(pin "3"
-		)
-		(instances
-			(project "rc_keychain"
-				(path "/c6cb5a1d-9f97-4766-8582-a9e93ed049e4/24c06676-89c1-498c-8350-9d02668ef39e"
-					(reference "SW1")
-					(unit 1)
-				)
-			)
-		)
-	)
-	(symbol
 		(lib_id "Device:C_Small")
 		(at 265.43 35.56 0)
@@
 	(symbol
 		(lib_id "Device:R_Small")
-		(at 166.37 74.93 0)
+		(at 165.1 72.39 0)
 		(unit 1)
 		(exclude_from_sim no)
@@
 		(fields_autoplaced yes)
 		(property "Reference" "R17"
-			(at 168.91 73.6599 0)
+			(at 167.64 71.1199 0)
 			(effects
 				(font
@@
 		)
 		(property "Value" "5.1k"
-			(at 168.91 76.1999 0)
+			(at 167.64 73.6599 0)
 			(effects
 				(font
@@
 		)
 		(property "Footprint" "Resistor_SMD:R_0402_1005Metric"
-			(at 166.37 74.93 0)
+			(at 165.1 72.39 0)
 			(effects
 				(font
@@
 		)
 		(property "Datasheet" "~"
-			(at 166.37 74.93 0)
+			(at 165.1 72.39 0)
 			(effects
 				(font
@@
 		)
 		(property "Description" "Resistor, small symbol"
-			(at 166.37 74.93 0)
+			(at 165.1 72.39 0)
 			(effects
 				(font
@@
 		)
 		(property "LCSC Part" "C25905"
-			(at 166.37 74.93 0)
+			(at 165.1 72.39 0)
 			(effects
 				(font
@@
 		)
 		(property "CREATOR" ""
-			(at 166.37 74.93 0)
+			(at 165.1 72.39 0)
 			(effects
 				(font
@@
 		)
 		(property "MAXIMUM_PACKAGE_HEIGHT" ""
-			(at 166.37 74.93 0)
+			(at 165.1 72.39 0)
 			(effects
 				(font
@@
 		)
 		(property "PARTREV" ""
-			(at 166.37 74.93 0)
+			(at 165.1 72.39 0)
 			(effects
 				(font
@@
 		)
 		(property "VERIFIER" ""
-			(at 166.37 74.93 0)
+			(at 165.1 72.39 0)
 			(effects
 				(font
@@
 		)
 		(property "AVAILABILITY" ""
-			(at 166.37 74.93 0)
+			(at 165.1 72.39 0)
 			(effects
 				(font
@@
 		)
 		(property "DESCRIPTION" ""
-			(at 166.37 74.93 0)
+			(at 165.1 72.39 0)
 			(effects
 				(font
@@
 		)
 		(property "MANUFACTURER" ""
-			(at 166.37 74.93 0)
+			(at 165.1 72.39 0)
 			(effects
 				(font
@@
 		)
 		(property "PACKAGE" ""
-			(at 166.37 74.93 0)
+			(at 165.1 72.39 0)
 			(effects
 				(font
@@
 		)
 		(property "PRICE" ""
-			(at 166.37 74.93 0)
+			(at 165.1 72.39 0)
 			(effects
 				(font
@@
 		)
 		(property "STANDARD" ""
-			(at 166.37 74.93 0)
+			(at 165.1 72.39 0)
 			(effects
 				(font
@@
 					(unit 1)
 				)
+			)
+		)
+	)
+	(symbol
+		(lib_id "HX3x4x2-2P-1:HX3X4X2-2P-1.6NTACTILESWITCH")
+		(at 179.07 78.74 0)
+		(unit 1)
+		(exclude_from_sim no)
+		(in_bom yes)
+		(on_board yes)
+		(dnp no)
+		(fields_autoplaced yes)
+		(property "Reference" "SW1"
+			(at 179.07 73.66 0)
+			(effects
+				(font
+					(size 1.27 1.27)
+				)
+			)
+		)
+		(property "Value" "HX 3X4X2-2P-1.6N"
+			(at 179.07 76.2 0)
+			(effects
+				(font
+					(size 1.27 1.27)
+				)
+			)
+		)
+		(property "Footprint" "HX3x4x2-2P-1:KEY-SMD_L4.0-W3.0-LS4.9-1"
+			(at 179.07 87.63 0)
+			(effects
+				(font
+					(size 1.27 1.27)
+				)
+				(hide yes)
+			)
+		)
+		(property "Datasheet" "https://www.lcsc.com/datasheet/C49234124.pdf"
+			(at 179.07 90.17 0)
+			(effects
+				(font
+					(size 1.27 1.27)
+				)
+				(hide yes)
+			)
+		)
+		(property "Description" ""
+			(at 179.07 78.74 0)
+			(effects
+				(font
+					(size 1.27 1.27)
+				)
+				(hide yes)
+			)
+		)
+		(property "Manufacturer" "hanxia(韩下)"
+			(at 179.07 92.71 0)
+			(effects
+				(font
+					(size 1.27 1.27)
+				)
+				(hide yes)
+			)
+		)
+		(property "MPN" "HX 3x4x2-2P-1.6N TACTILE SWITCH"
+			(at 179.07 95.25 0)
+			(effects
+				(font
+					(size 1.27 1.27)
+				)
+				(hide yes)
+			)
+		)
+		(property "LCSC Part" "C49234124"
+			(at 179.07 97.79 0)
+			(effects
+				(font
+					(size 1.27 1.27)
+				)
+				(hide yes)
+			)
+		)
+		(pin "2"
+		)
+		(pin "1"
+		)
+		(instances
+			(project ""
+				(path "/c6cb5a1d-9f97-4766-8582-a9e93ed049e4/24c06676-89c1-498c-8350-9d02668ef39e"
+					(reference "SW1")
+					(unit 1)
+				)

Commit message: progress before restarting bigtime
Other:
- moved on the sheet: D5
Changed lines of the file:
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@@
 	(wire
 		(pts
-			(xy 214.63 138.43) (xy 215.9 138.43)
+			(xy 214.63 138.43) (xy 217.17 138.43)
 		)
 		(stroke
@@
 	(wire
 		(pts
-			(xy 223.52 138.43) (xy 228.6 138.43)
+			(xy 224.79 138.43) (xy 228.6 138.43)
 		)
 		(stroke
@@
 	(symbol
 		(lib_id "Device:LED")
-		(at 219.71 138.43 180)
+		(at 220.98 138.43 180)
 		(unit 1)
 		(exclude_from_sim no)
@@
 		(dnp no)
 		(property "Reference" "D5"
-			(at 221.2975 130.81 0)
+			(at 220.98 132.334 0)
 			(effects
 				(font
@@
 		)
 		(property "Value" "KT-0805G"
-			(at 221.2975 133.35 0)
+			(at 220.98 134.62 0)
 			(effects
 				(font
@@
 		)
 		(property "Footprint" "Diode_SMD:D_0805_2012Metric"
-			(at 219.71 138.43 0)
+			(at 220.98 138.43 0)
 			(effects
 				(font
@@
 		)
 		(property "Datasheet" "~"
-			(at 219.71 138.43 0)
+			(at 220.98 138.43 0)
 			(effects
 				(font
@@
 		)
 		(property "Description" "Light emitting diode"
-			(at 219.71 138.43 0)
+			(at 220.98 138.43 0)
 			(effects
 				(font
@@
 		)
 		(property "Sim.Pins" "1=K 2=A"
-			(at 219.71 138.43 0)
+			(at 220.98 138.43 0)
 			(effects
 				(font
@@
 		)
 		(property "LCSC Part" "C2297"
-			(at 219.71 138.43 0)
+			(at 220.98 138.43 0)
 			(effects
 				(font

Commit message: progress before finagling
Connections:
- net +3V3_G2: now also C27.1, L4.1, U9.5 (VIN)
- net VBAT: no longer C27.1, L4.1, U9.5 (VIN)
Changed lines of the file:
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@@
+	)
+	(symbol
+		(lib_id "custom_syms:+3V3_G2")
+		(at 96.52 151.13 0)
+		(unit 1)
+		(exclude_from_sim no)
+		(in_bom yes)
+		(on_board yes)
+		(dnp no)
+		(property "Reference" "#PWR011"
+			(at 96.52 154.94 0)
+			(effects
+				(font
+					(size 1.27 1.27)
+				)
+				(hide yes)
+			)
+		)
+		(property "Value" "+3V3_G2"
+			(at 96.52 147.066 0)
+			(effects
+				(font
+					(size 1.27 1.27)
+				)
+			)
+		)
+		(property "Footprint" ""
+			(at 96.52 151.13 0)
+			(effects
+				(font
+					(size 1.27 1.27)
+				)
+				(hide yes)
+			)
+		)
+		(property "Datasheet" ""
+			(at 96.52 151.13 0)
+			(effects
+				(font
+					(size 1.27 1.27)
+				)
+				(hide yes)
+			)
+		)
+		(property "Description" "Power symbol creates a global label with name \"+3V3_G2\""
+			(at 96.52 151.13 0)
+			(effects
+				(font
+					(size 1.27 1.27)
+				)
+				(hide yes)
+			)
+		)
+		(pin "1"
+		)
+		(instances
+			(project ""
+				(path "/c6cb5a1d-9f97-4766-8582-a9e93ed049e4/24c06676-89c1-498c-8350-9d02668ef39e"
+					(reference "#PWR011")
+					(unit 1)
+				)
+			)
+		)
 	)
 	(symbol
@@
 					(unit 1)
 				)
-			)
-		)
-	)
-	(symbol
-		(lib_id "custom_syms:VBAT")
-		(at 96.52 151.13 0)
-		(unit 1)
-		(exclude_from_sim no)
-		(in_bom yes)
-		(on_board yes)
-		(dnp no)
-		(fields_autoplaced yes)
-		(property "Reference" "#PWR073"
-			(at 96.52 154.94 0)
-			(effects
-				(font
-					(size 1.27 1.27)
-				)
-				(hide yes)
-			)
-		)
-		(property "Value" "VBAT"
-			(at 96.52 146.05 0)
-			(effects
-				(font
-					(size 1.27 1.27)
-				)
-			)
-		)
-		(property "Footprint" ""
-			(at 96.52 151.13 0)
-			(effects
-				(font
-					(size 1.27 1.27)
-				)
-				(hide yes)
-			)
-		)
-		(property "Datasheet" ""
-			(at 96.52 151.13 0)
-			(effects
-				(font
-					(size 1.27 1.27)
-				)
-				(hide yes)
-			)
-		)
-		(property "Description" "Power symbol creates a global label with name \"VBAT\""
-			(at 96.52 151.13 0)
-			(effects
-				(font
-					(size 1.27 1.27)
-				)
-				(hide yes)
-			)
-		)
-		(pin "1"
-		)
-		(instances
-			(project ""
-				(path "/c6cb5a1d-9f97-4766-8582-a9e93ed049e4/24c06676-89c1-498c-8350-9d02668ef39e"
-					(reference "#PWR073")
-					(unit 1)
-				)

Commit message: progress mid-finagling
Parts:
- removed SW1: HX 3X4X2-2P-1.6N, HX3x4x2-2P-1:KEY-SMD_L4.0-W3.0-LS4.9-1, symbol HX3x4x2-2P-1:HX3X4X2-2P-1.6NTACTILESWITCH
- added SW2: HX-B3U-1000P-1.6N, HX-B3U-1000P-1:SW-SMD_2P-L3.0-W2.5-LS4.0, symbol HX-B3U-1000P-1:HX-B3U-1000P-1.6N
Connections:
- net BUTTON: now also SW2.2
- net at R17.2: now also SW2.1
Other:
- moved on the sheet: R17
Changed lines of the file:
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@@
 	(wire
 		(pts
-			(xy 184.15 80.01) (xy 189.23 80.01)
+			(xy 185.42 80.01) (xy 189.23 80.01)
 		)
 		(stroke
@@
 	(wire
 		(pts
-			(xy 165.1 80.01) (xy 173.99 80.01)
+			(xy 106.68 143.51) (xy 114.3 143.51)
 		)
 		(stroke
@@
 	(wire
 		(pts
-			(xy 106.68 143.51) (xy 114.3 143.51)
+			(xy 163.83 80.01) (xy 175.26 80.01)
 		)
 		(stroke
@@
 	(wire
 		(pts
-			(xy 165.1 74.93) (xy 165.1 80.01)
+			(xy 163.83 74.93) (xy 163.83 80.01)
 		)
 		(stroke
@@
 	(symbol
 		(lib_id "power:+3V3")
-		(at 165.1 69.85 0)
+		(at 163.83 69.85 0)
 		(unit 1)
 		(exclude_from_sim no)
@@
 		(fields_autoplaced yes)
 		(property "Reference" "#PWR082"
-			(at 165.1 73.66 0)
+			(at 163.83 73.66 0)
 			(effects
 				(font
@@
 		)
 		(property "Value" "+3V3"
-			(at 165.1 64.77 0)
+			(at 163.83 64.77 0)
 			(effects
 				(font
@@
 		)
 		(property "Footprint" ""
-			(at 165.1 69.85 0)
+			(at 163.83 69.85 0)
 			(effects
 				(font
@@
 		)
 		(property "Datasheet" ""
-			(at 165.1 69.85 0)
+			(at 163.83 69.85 0)
 			(effects
 				(font
@@
 		)
 		(property "Description" "Power symbol creates a global label with name \"+3V3\""
-			(at 165.1 69.85 0)
+			(at 163.83 69.85 0)
 			(effects
 				(font
@@
 	)
 	(symbol
+		(lib_id "HX-B3U-1000P-1:HX-B3U-1000P-1.6N")
+		(at 180.34 78.74 0)
+		(unit 1)
+		(exclude_from_sim no)
+		(in_bom yes)
+		(on_board yes)
+		(dnp no)
+		(fields_autoplaced yes)
+		(property "Reference" "SW2"
+			(at 180.34 73.66 0)
+			(effects
+				(font
+					(size 1.27 1.27)
+				)
+			)
+		)
+		(property "Value" "HX-B3U-1000P-1.6N"
+			(at 180.34 76.2 0)
+			(effects
+				(font
+					(size 1.27 1.27)
+				)
+			)
+		)
+		(property "Footprint" "HX-B3U-1000P-1:SW-SMD_2P-L3.0-W2.5-LS4.0"
+			(at 180.34 87.63 0)
+			(effects
+				(font
+					(size 1.27 1.27)
+				)
+				(hide yes)
+			)
+		)
+		(property "Datasheet" "https://www.lcsc.com/datasheet/C49234121.pdf"
+			(at 180.34 90.17 0)
+			(effects
+				(font
+					(size 1.27 1.27)
+				)
+				(hide yes)
+			)
+		)
+		(property "Description" ""
+			(at 180.34 78.74 0)
+			(effects
+				(font
+					(size 1.27 1.27)
+				)
+				(hide yes)
+			)
+		)
+		(property "Manufacturer" "hanxia(韩下)"
+			(at 180.34 92.71 0)
+			(effects
+				(font
+					(size 1.27 1.27)
+				)
+				(hide yes)
+			)
+		)
+		(property "MPN" "HX-B3U-1000P-1.6N"
+			(at 180.34 95.25 0)
+			(effects
+				(font
+					(size 1.27 1.27)
+				)
+				(hide yes)
+			)
+		)
+		(property "LCSC Part" "C49234121"
+			(at 180.34 97.79 0)
+			(effects
+				(font
+					(size 1.27 1.27)
+				)
+				(hide yes)
+			)
+		)
+		(pin "1"
+		)
+		(pin "2"
+		)
+		(instances
+			(project ""
+				(path "/c6cb5a1d-9f97-4766-8582-a9e93ed049e4/24c06676-89c1-498c-8350-9d02668ef39e"
+					(reference "SW2")
+					(unit 1)
+				)
+			)
+		)
+	)
+	(symbol
 		(lib_id "power:GND")
 		(at 87.63 40.64 90)
@@
 	(symbol
 		(lib_id "Device:R_Small")
-		(at 165.1 72.39 0)
+		(at 163.83 72.39 0)
 		(unit 1)
 		(exclude_from_sim no)
@@
 		(fields_autoplaced yes)
 		(property "Reference" "R17"
-			(at 167.64 71.1199 0)
+			(at 166.37 71.1199 0)
 			(effects
 				(font
@@
 		)
 		(property "Value" "5.1k"
-			(at 167.64 73.6599 0)
+			(at 166.37 73.6599 0)
 			(effects
 				(font
@@
 		)
 		(property "Footprint" "Resistor_SMD:R_0402_1005Metric"
-			(at 165.1 72.39 0)
+			(at 163.83 72.39 0)
 			(effects
 				(font
@@
 		)
 		(property "Datasheet" "~"
-			(at 165.1 72.39 0)
+			(at 163.83 72.39 0)
 			(effects
 				(font
@@
 		)
 		(property "Description" "Resistor, small symbol"
-			(at 165.1 72.39 0)
+			(at 163.83 72.39 0)
 			(effects
 				(font
@@
 		)
 		(property "LCSC Part" "C25905"
-			(at 165.1 72.39 0)
+			(at 163.83 72.39 0)
 			(effects
 				(font
@@
 		)
 		(property "CREATOR" ""
-			(at 165.1 72.39 0)
+			(at 163.83 72.39 0)
 			(effects
 				(font
@@
 		)
 		(property "MAXIMUM_PACKAGE_HEIGHT" ""
-			(at 165.1 72.39 0)
+			(at 163.83 72.39 0)
 			(effects
 				(font
@@
 		)
 		(property "PARTREV" ""
-			(at 165.1 72.39 0)
+			(at 163.83 72.39 0)
 			(effects
 				(font
@@
 		)
 		(property "VERIFIER" ""
-			(at 165.1 72.39 0)
+			(at 163.83 72.39 0)
 			(effects
 				(font
@@
 		)
 		(property "AVAILABILITY" ""
-			(at 165.1 72.39 0)
+			(at 163.83 72.39 0)
 			(effects
 				(font
@@
 		)
 		(property "DESCRIPTION" ""
-			(at 165.1 72.39 0)
+			(at 163.83 72.39 0)
 			(effects
 				(font
@@
 		)
 		(property "MANUFACTURER" ""
-			(at 165.1 72.39 0)
+			(at 163.83 72.39 0)
 			(effects
 				(font
@@
 		)
 		(property "PACKAGE" ""
-			(at 165.1 72.39 0)
+			(at 163.83 72.39 0)
 			(effects
 				(font
@@
 		)
 		(property "PRICE" ""
-			(at 165.1 72.39 0)
+			(at 163.83 72.39 0)
 			(effects
 				(font
@@
 		)
 		(property "STANDARD" ""
-			(at 165.1 72.39 0)
+			(at 163.83 72.39 0)
 			(effects
 				(font
@@
 					(unit 1)
 				)
-			)
-		)
-	)
-	(symbol
-		(lib_id "HX3x4x2-2P-1:HX3X4X2-2P-1.6NTACTILESWITCH")
-		(at 179.07 78.74 0)
-		(unit 1)
-		(exclude_from_sim no)
-		(in_bom yes)
-		(on_board yes)
-		(dnp no)
-		(fields_autoplaced yes)
-		(property "Reference" "SW1"
-			(at 179.07 73.66 0)
-			(effects
-				(font
-					(size 1.27 1.27)
-				)
-			)
-		)
-		(property "Value" "HX 3X4X2-2P-1.6N"
-			(at 179.07 76.2 0)
-			(effects
-				(font
-					(size 1.27 1.27)
-				)
-			)
-		)
-		(property "Footprint" "HX3x4x2-2P-1:KEY-SMD_L4.0-W3.0-LS4.9-1"
-			(at 179.07 87.63 0)
-			(effects
-				(font
-					(size 1.27 1.27)
-				)
-				(hide yes)
-			)
-		)
-		(property "Datasheet" "https://www.lcsc.com/datasheet/C49234124.pdf"
-			(at 179.07 90.17 0)
-			(effects
-				(font
-					(size 1.27 1.27)
-				)
-				(hide yes)
-			)
-		)
-		(property "Description" ""
-			(at 179.07 78.74 0)
-			(effects
-				(font
-					(size 1.27 1.27)
-				)
-				(hide yes)
-			)
-		)
-		(property "Manufacturer" "hanxia(韩下)"
-			(at 179.07 92.71 0)
-			(effects
-				(font
-					(size 1.27 1.27)
-				)
-				(hide yes)
-			)
-		)
-		(property "MPN" "HX 3x4x2-2P-1.6N TACTILE SWITCH"
-			(at 179.07 95.25 0)
-			(effects
-				(font
-					(size 1.27 1.27)
-				)
-				(hide yes)
-			)
-		)
-		(property "LCSC Part" "C49234124"
-			(at 179.07 97.79 0)
-			(effects
-				(font
-					(size 1.27 1.27)
-				)
-				(hide yes)
-			)
-		)
-		(pin "2"
-		)
-		(pin "1"
-		)
-		(instances
-			(project ""
-				(path "/c6cb5a1d-9f97-4766-8582-a9e93ed049e4/24c06676-89c1-498c-8350-9d02668ef39e"
-					(reference "SW1")
-					(unit 1)
-				)

Commit message: huge progress
Parts:
- removed C34: 10uF, Capacitor_SMD:C_0402_1005Metric, symbol Device:C_Small
- removed U10: LIS3DH, Package_LGA:LGA-16_3x3mm_P0.5mm_LayoutBorder3x5y, symbol Sensor_Motion:LIS3DH
- removed U9: TPS61040DBV, Package_TO_SOT_SMD:SOT-23-5, symbol Regulator_Switching:TPS61040DBV
- added C1: 2.2uF, Capacitor_SMD:C_0402_1005Metric, symbol Device:C_Small
- added U10: QMC6309, QMC6309:X1-WLB0808-4_L0.8-W0.8-P0.40-TL, symbol QMC6309:QMC6309
- added U11: TPS61040DRV, Package_SON:WSON-6-1EP_2x2mm_P0.65mm_EP1x1.6mm, symbol Regulator_Switching:TPS61040DRV
- added U14: LSM6DS3, Package_LGA:LGA-14_3x2.5mm_P0.5mm_LayoutBorder3x4y, symbol Sensor_Motion:LSM6DS3
- D1: footprint Diode_SMD:D_SOD-123 -> Diode_SMD:D_SOD-323; LCSC Part C5563735 -> C49238168
- L4: footprint Inductor_SMD:L_1008_2520Metric -> FTC201610S4R7MBCA:IND-SMD_L2.0-W1.6-B; LCSC Part C5159366 -> C5832346
Connections:
- net +3V3: now also C1.1, U10.A1 (VSS), U14.12 (CS), U14.5 (VDDIO), U14.8 (VDD)
- net +3V3_G2: now also U11.2 (VIN), U11.3 (EN)
- net ACC_INT: now also U14.4 (INT1)
- net GND: now also C1.2, U10.B1 (VDD), U11.1 (GND), U14.1 (SDO/SA0), U14.2 (SDX), U14.3 (SCX), U14.6 (GND), U14.7 (GND)
- net SCL: now also U10.A2 (SCL), U14.13 (SCL)
- net SDA: now also U10.B2 (SDA), U14.14 (SDA)
- net at C29.2, R15.1, R16.2: now also U11.4 (FB)
- net at D1.2 (A), L4.2: now also U11.6 (SW)
- no-connect marks 5 -> 2
Other:
- moved on the sheet: C33, C35

Commit message: first draft of final board
Other:
- moved on the sheet: D5, R1
Changed lines of the file:
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@@
 	(wire
 		(pts
-			(xy 214.63 138.43) (xy 217.17 138.43)
+			(xy 209.55 132.08) (xy 212.09 132.08)
 		)
 		(stroke
@@
 	(wire
 		(pts
-			(xy 224.79 138.43) (xy 228.6 138.43)
+			(xy 219.71 132.08) (xy 223.52 132.08)
 		)
 		(stroke
@@
 	(wire
 		(pts
-			(xy 236.22 140.97) (xy 236.22 138.43)
+			(xy 231.14 134.62) (xy 231.14 132.08)
 		)
 		(stroke
@@
 	(wire
 		(pts
-			(xy 236.22 138.43) (xy 233.68 138.43)
+			(xy 231.14 132.08) (xy 228.6 132.08)
 		)
 		(stroke
@@
 	(global_label "LED_DAT"
 		(shape input)
-		(at 214.63 138.43 180)
+		(at 209.55 132.08 180)
 		(fields_autoplaced yes)
 		(effects
@@
 		)
 		(property "Intersheetrefs" "${INTERSHEET_REFS}"
-			(at 203.9039 138.43 0)
+			(at 198.8239 132.08 0)
 			(effects
 				(font
@@
 	(symbol
 		(lib_id "Device:R_Small")
-		(at 231.14 138.43 270)
+		(at 226.06 132.08 270)
 		(unit 1)
 		(exclude_from_sim no)
@@
 		(fields_autoplaced yes)
 		(property "Reference" "R1"
-			(at 231.14 133.35 90)
+			(at 226.06 127 90)
 			(effects
 				(font
@@
 		)
 		(property "Value" "100"
-			(at 231.14 135.89 90)
+			(at 226.06 129.54 90)
 			(effects
 				(font
@@
 		)
 		(property "Footprint" "Resistor_SMD:R_0402_1005Metric"
-			(at 231.14 138.43 0)
+			(at 226.06 132.08 0)
 			(effects
 				(font
@@
 		)
 		(property "Datasheet" "~"
-			(at 231.14 138.43 0)
+			(at 226.06 132.08 0)
 			(effects
 				(font
@@
 		)
 		(property "Description" "Resistor, small symbol"
-			(at 231.14 138.43 0)
+			(at 226.06 132.08 0)
 			(effects
 				(font
@@
 	(symbol
 		(lib_id "power:GND")
-		(at 236.22 140.97 0)
+		(at 231.14 134.62 0)
 		(unit 1)
 		(exclude_from_sim no)
@@
 		(fields_autoplaced yes)
 		(property "Reference" "#PWR08"
-			(at 236.22 147.32 0)
+			(at 231.14 140.97 0)
 			(effects
 				(font
@@
 		)
 		(property "Value" "GND"
-			(at 236.22 146.05 0)
+			(at 231.14 139.7 0)
 			(effects
 				(font
@@
 		)
 		(property "Footprint" ""
-			(at 236.22 140.97 0)
+			(at 231.14 134.62 0)
 			(effects
 				(font
@@
 		)
 		(property "Datasheet" ""
-			(at 236.22 140.97 0)
+			(at 231.14 134.62 0)
 			(effects
 				(font
@@
 		)
 		(property "Description" "Power symbol creates a global label with name \"GND\" , ground"
-			(at 236.22 140.97 0)
+			(at 231.14 134.62 0)
 			(effects
 				(font
@@
 	(symbol
 		(lib_id "Device:LED")
-		(at 220.98 138.43 180)
+		(at 215.9 132.08 180)
 		(unit 1)
 		(exclude_from_sim no)
@@
 		(dnp no)
 		(property "Reference" "D5"
-			(at 220.98 132.334 0)
+			(at 215.9 125.984 0)
 			(effects
 				(font
@@
 		)
 		(property "Value" "KT-0805G"
-			(at 220.98 134.62 0)
+			(at 215.9 128.27 0)
 			(effects
 				(font
@@
 		)
 		(property "Footprint" "Diode_SMD:D_0805_2012Metric"
-			(at 220.98 138.43 0)
+			(at 215.9 132.08 0)
 			(effects
 				(font
@@
 		)
 		(property "Datasheet" "~"
-			(at 220.98 138.43 0)
+			(at 215.9 132.08 0)
 			(effects
 				(font
@@
 		)
 		(property "Description" "Light emitting diode"
-			(at 220.98 138.43 0)
+			(at 215.9 132.08 0)
 			(effects
 				(font
@@
 		)
 		(property "Sim.Pins" "1=K 2=A"
-			(at 220.98 138.43 0)
+			(at 215.9 132.08 0)
 			(effects
 				(font
@@
 		)
 		(property "LCSC Part" "C2297"
-			(at 220.98 138.43 0)
+			(at 215.9 132.08 0)
 			(effects
 				(font
