File: interface.kicad_sch (KiCad schematic)
At the start: 27 parts, among them J5 5034801200, SW2 HX-B3U-1000P-1.6N, U10 QMC6309, U11 TPS61040DRV, U14 LSM6DS3, U8 DRV2603RUNT

Commit message: final fixups before prod
Parts:
- removed TP28: 9V, TestPoint:TestPoint_Pad_D1.0mm, symbol Connector:TestPoint
- removed TP37: BUTTON, TestPoint:TestPoint_Pad_D1.0mm, symbol Connector:TestPoint
- C28: renamed from C30; LCSC Part C1705 -> C19666
- C31: renamed from C1; LCSC Part (none) -> C12530
- R19: renamed from R1; LCSC Part (none) -> C25076
- renumbered C27 to C24, C28 to C25, C29 to C27, C31 to C29, C33 to C30, C35 to C32, D1 to D2, D5 to D3, J5 to J4, SW2 to SW1, U14 to U10, U10 to U11, U11 to U9
