File: power.kicad_sch (KiCad schematic)
At the start: 23 parts, among them U1 SF32LB525UC6

Commit message: layout progress
Parts:
- C10, C19: footprint Capacitor_SMD:C_0402_1005Metric -> Capacitor_SMD:C_0201_0603Metric; LCSC Part C23733 -> (none)
- C13, C14: footprint Capacitor_SMD:C_0201_1005Metric -> Capacitor_SMD:C_0201_0603Metric
Changed lines of the file:
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@@
 			)
 		)
-		(property "Footprint" "Capacitor_SMD:C_0402_1005Metric"
+		(property "Footprint" "Capacitor_SMD:C_0201_0603Metric"
 			(at 195.58 121.92 0)
 			(effects
@@
 			)
 		)
-		(property "LCSC Part" "C23733"
+		(property "LCSC Part" ""
 			(at 195.58 121.92 90)
 			(effects
@@
 			)
 		)
-		(property "Footprint" "Capacitor_SMD:C_0402_1005Metric"
+		(property "Footprint" "Capacitor_SMD:C_0201_0603Metric"
 			(at 123.19 142.24 0)
 			(effects
@@
 			)
 		)
-		(property "LCSC Part" "C23733"
+		(property "LCSC Part" ""
 			(at 123.19 142.24 0)
 			(effects
@@
 			)
 		)
-		(property "Footprint" "Capacitor_SMD:C_0201_1005Metric"
+		(property "Footprint" "Capacitor_SMD:C_0201_0603Metric"
 			(at 190.5 104.14 0)
 			(effects
@@
 			)
 		)
-		(property "Footprint" "Capacitor_SMD:C_0201_1005Metric"
+		(property "Footprint" "Capacitor_SMD:C_0201_0603Metric"
 			(at 190.5 109.22 0)
 			(effects

Commit message: huge progress
Changed lines of the file:
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@@
 		(color 0 0 0 0)
+	)
+	(bus_entry
+		(at 190.5 143.51)
+		(size 2.54 2.54)
+		(stroke
+			(width 0)
+			(type default)
+		)
 	)
 	(wire

Commit message: final fixups before prod
Parts:
- removed TP10: GND, TestPoint:TestPoint_Pad_D1.0mm, symbol Connector:TestPoint
- removed TP11: 3V3, TestPoint:TestPoint_Pad_D1.0mm, symbol Connector:TestPoint
- removed TP24: VBUS, TestPoint:TestPoint_Pad_D1.0mm, symbol Connector:TestPoint
- removed TP26: 3V3_G1, TestPoint:TestPoint_Pad_D1.0mm, symbol Connector:TestPoint
- removed TP27: 3V3_G2, TestPoint:TestPoint_Pad_D1.0mm, symbol Connector:TestPoint
- removed TP9: VBAT, TestPoint:TestPoint_Pad_D1.0mm, symbol Connector:TestPoint
- C15: renamed from C19; LCSC Part (none) -> C335103
- C6: renamed from C10; LCSC Part (none) -> C335103
- C7: renamed from C11; LCSC Part C77762 -> C335106
- renumbered C14 to C10, C15 to C11, C16 to C12, C17 to C13, C18 to C14, C20 to C16, C21 to C17, C8 to C4, C9 to C5, C12 to C8, C13 to C9
